Commit message: update urdf

File: orthrus_sim/orthrus_gazebo/models/orthrus/urdf/orthrus.urdf (robot description, URDF)
Before this commit: robot gazebo1, 13 links, 12 joints
Links:
- link body: mass 10 -> 7
- link hip_LB: mass 1 -> 0.7
- link hip_LF: mass 1 -> 0.7
- link hip_RB: mass 1 -> 0.7
- link hip_RF: mass 1 -> 0.7
- link leg2_LB: mass 1 -> 0.2
- link leg2_LF: mass 1 -> 0.2
- link leg2_RB: mass 1 -> 0.2
- link leg2_RF: mass 1 -> 0.2

File: orthrus_sim/orthrus_gazebo/models/orthrus/urdf/orthrus.urdf.xacro (robot description, xacro)
@@ -27,7 +27,6 @@
     </collision>
     <inertial>
-      <origin xyz="-0.10 0.1385 -0.05" rpy="${pi/2} 0 0" />
       <mass value="7"/>
-      <inertia ixx="4.9950395" ixy="0" ixz="0" iyy="6.4183150" iyz="0" izz="2.4616377" />
+      <inertia ixx="4.9950395" ixy="0" ixz="0" iyy="2.4616377" iyz="0" izz="6.4183150" />
     </inertial>
   </link>
@@ -47,5 +46,8 @@
         </geometry>
       </collision>
-      <xacro:default_inertial mass="1"/>
+      <inertial>
+        <mass value="0.7"/>
+        <inertia ixx="0.0904981" ixy="0" ixz="-0.0000480" iyy=" 0.0917319" iyz="0" izz="0.0857923" />
+      </inertial>
     </link>
     <joint name="hip_${prefix}_joint" type="revolute">
@@ -53,5 +55,5 @@
       <parent link="body"/>
       <child link="hip_${prefix}"/>
-      <dynamics damping="0.5" friction="0.1"/>
+      <dynamics damping="0.1" friction="0.01"/>
       <limit effort="35.0" lower="-${pi/2}" upper="${pi/2}" velocity="${pi}"/>
       <xacro:if value="${prefix == 'LF'}">
@@ -88,5 +90,8 @@
         </geometry>
       </collision>
-      <xacro:default_inertial mass="1"/>
+      <inertial>
+        <mass value="1"/>
+        <inertia ixx="0.4329464" ixy="-0.0830239" ixz=" -0.0000001" iyy="0.1503071" iyz="0.0000001" izz="0.4817994" />
+      </inertial>
     </link>
     <joint name="leg1_${prefix}_joint" type="revolute">
@@ -94,5 +99,5 @@
       <parent link="hip_${prefix}"/>
       <child link="leg1_${prefix}"/>
-      <dynamics damping="0.5" friction="0.1"/>
+      <dynamics damping="0.1" friction="0.01"/>
       <limit effort="35.0" lower="-${pi*2/3}" upper="${pi*2/3}" velocity="${pi}"/>
       <xacro:if value="${prefix == 'LF'}">
@@ -129,5 +134,8 @@
         </geometry>
       </collision>
-      <xacro:default_inertial mass="1"/>
+      <inertial>
+        <mass value="0.2"/>
+        <inertia ixx="0.4201680" ixy="0" ixz="0" iyy="0.4196489" iyz="0" izz="0.0031965" />
+      </inertial>
     </link>
     <joint name="leg2_${prefix}_joint" type="revolute">
@@ -135,5 +143,5 @@
       <parent link="leg1_${prefix}"/>
       <child link="leg2_${prefix}"/>
-      <dynamics damping="0.5" friction="0.1"/>
+      <dynamics damping="0.1" friction="0.01"/>
       <xacro:if value="${prefix == 'LF'}">
         <origin xyz="0.035 -0.18 0" rpy="${pi*2/3} 0 0" />

Commit message: update

File: orthrus_sim/orthrus_gazebo/models/orthrus/urdf/orthrus.urdf (robot description, URDF)
Before this commit: robot orthrus, 13 links, 12 joints
Links:
- link body: geometry collision mesh filename=file:////home/evence/code_file/ros2_ws/orthrus/install/orth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; visual mesh filename=file:////home/evence/code_file/ros2_ws/orthrus/install/orth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
- link hip_LB: geometry collision mesh filename=file:////home/evence/code_file/ros2_ws/orthrus/install/orth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; visual mesh filename=file:////home/evence/code_file/ros2_ws/orthrus/install/orth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
- link hip_LF: geometry collision mesh filename=file:////home/evence/code_file/ros2_ws/orthrus/install/orth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; visual mesh filename=file:////home/evence/code_file/ros2_ws/orthrus/install/orth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
- link hip_RB: geometry collision mesh filename=file:////home/evence/code_file/ros2_ws/orthrus/install/orth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; visual mesh filename=file:////home/evence/code_file/ros2_ws/orthrus/install/orth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
- link hip_RF: geometry collision mesh filename=file:////home/evence/code_file/ros2_ws/orthrus/install/orth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; visual mesh filename=file:////home/evence/code_file/ros2_ws/orthrus/install/orth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
- link leg1_LB: geometry collision mesh filename=file:////home/evence/code_file/ros2_ws/orthrus/install/orth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; visual mesh filename=file:////home/evence/code_file/ros2_ws/orthrus/install/orth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
- link leg1_LF: geometry collision mesh filename=file:////home/evence/code_file/ros2_ws/orthrus/install/orth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; visual mesh filename=file:////home/evence/code_file/ros2_ws/orthrus/install/orth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
- link leg1_RB: geometry collision mesh filename=file:////home/evence/code_file/ros2_ws/orthrus/install/orth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; visual mesh filename=file:////home/evence/code_file/ros2_ws/orthrus/install/orth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
- link leg1_RF: geometry collision mesh filename=file:////home/evence/code_file/ros2_ws/orthrus/install/orth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; visual mesh filename=file:////home/evence/code_file/ros2_ws/orthrus/install/orth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
- link leg2_LB: geometry collision mesh filename=file:////home/evence/code_file/ros2_ws/orthrus/install/orth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; visual mesh filename=file:////home/evence/code_file/ros2_ws/orthrus/install/orth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
- link leg2_LF: geometry collision mesh filename=file:////home/evence/code_file/ros2_ws/orthrus/install/orth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; visual mesh filename=file:////home/evence/code_file/ros2_ws/orthrus/install/orth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
- link leg2_RB: geometry collision mesh filename=file:////home/evence/code_file/ros2_ws/orthrus/install/orth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; visual mesh filename=file:////home/evence/code_file/ros2_ws/orthrus/install/orth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
- link leg2_RF: geometry collision mesh filename=file:////home/evence/code_file/ros2_ws/orthrus/install/orth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; visual mesh filename=file:////home/evence/code_file/ros2_ws/orthrus/install/orth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
