Commit message: update

File: orthrus_sim/orthrus_gazebo/models/orthrus/urdf/orthrus.urdf.xacro (robot description, xacro)
@@ -2,10 +2,4 @@
 <robot name="gazebo1"
   xmlns:xacro="http://ros.org/wiki/xacro">
-  <xacro:property name="width" value="0.2" />
-  <xacro:property name="leglen" value="0.6" />
-  <xacro:property name="polelen" value="0.2" />
-  <xacro:property name="bodylen" value="0.6" />
-  <xacro:property name="baselen" value="0.4" />
-  <xacro:property name="wheeldiam" value="0.07" />
   <xacro:property name="meshes_folder" value="$(find orthrus_gazebo)/models/orthrus/meshes" />
   <material name="blue">
@@ -18,10 +12,4 @@
     <color rgba="1 1 1 1"/>
   </material>
-  <xacro:macro name="default_inertial" params="mass">
-    <inertial>
-      <mass value="${mass}" />
-      <inertia ixx="1.0" ixy="0.0" ixz="0.0" iyy="1.0" iyz="0.0" izz="1.0" />
-    </inertial>
-  </xacro:macro>
   <link name="body">
     <visual>
@@ -38,5 +26,9 @@
       </geometry>
     </collision>
-    <xacro:default_inertial mass="10"/>
+    <inertial>
+      <origin xyz="-0.10 0.1385 -0.05" rpy="${pi/2} 0 0" />
+      <mass value="7"/>
+      <inertia ixx="4.9950395" ixy="0" ixz="0" iyy="6.4183150" iyz="0" izz="2.4616377" />
+    </inertial>
   </link>
   <xacro:macro name="hip" params="prefix">

Commit message: update

File: orthrus_sim/orthrus_gazebo/models/orthrus/urdf/orthrus.urdf.xacro (robot description, xacro)
@@ -168,7 +168,29 @@
   <xacro:macro name="ros2_hip_joint" params="prefix">
     <joint name="hip_${prefix}_joint">
-      <command_interface name="position">
-        <param name="min">-${pi/2}</param>
-        <param name="max">${pi/2}</param>
+      <command_interface name="effort">
+        <param name="min">-35</param>
+        <param name="max">35</param>
+      </command_interface>
+      <state_interface name="position"/>
+      <state_interface name="velocity"/>
+      <state_interface name="effort"/>
+    </joint>
+  </xacro:macro>
+  <xacro:macro name="ros2_leg1_joint" params="prefix">
+    <joint name="leg1_${prefix}_joint">
+      <command_interface name="effort">
+        <param name="min">-35</param>
+        <param name="max">35</param>
+      </command_interface>
+      <state_interface name="position"/>
+      <state_interface name="velocity"/>
+      <state_interface name="effort"/>
+    </joint>
+  </xacro:macro>
+  <xacro:macro name="ros2_leg2_joint" params="prefix">
+    <joint name="leg2_${prefix}_joint">
+      <command_interface name="effort">
+        <param name="min">-35</param>
+        <param name="max">35</param>
       </command_interface>
       <state_interface name="position"/>
@@ -182,4 +204,15 @@
     </hardware>
     <xacro:ros2_hip_joint prefix="RF"/>
+    <xacro:ros2_hip_joint prefix="LF"/>
+    <xacro:ros2_hip_joint prefix="RB"/>
+    <xacro:ros2_hip_joint prefix="LB"/>
+    <xacro:ros2_leg1_joint prefix="RF"/>
+    <xacro:ros2_leg1_joint prefix="LF"/>
+    <xacro:ros2_leg1_joint prefix="RB"/>
+    <xacro:ros2_leg1_joint prefix="LB"/>
+    <xacro:ros2_leg2_joint prefix="RF"/>
+    <xacro:ros2_leg2_joint prefix="LF"/>
+    <xacro:ros2_leg2_joint prefix="RB"/>
+    <xacro:ros2_leg2_joint prefix="LB"/>
   </ros2_control>
   <gazebo>

Commit message: update

File: orthrus_sim/orthrus_gazebo/models/orthrus/urdf/orthrus.urdf.xacro (robot description, xacro)
@@ -1,6 +1,7 @@
 <?xml version="1.0"?>
-<robot name="gazebo1"
+<robot name="orthrus"
   xmlns:xacro="http://ros.org/wiki/xacro">
-  <xacro:property name="meshes_folder" value="$(find orthrus_gazebo)/models/orthrus/meshes" />
+  <xacro:property name="meshes_folder" value="file:///$(find orthrus_gazebo)/models/orthrus/meshes" />
+  <!--<xacro:property name="meshes_folder" value="/home/evence/code_file/ros2_ws/orthrus/src/orthrus_ros2_pack/orthrus_sim/orthrus_gazebo/models/orthrus/meshes" />-->
   <material name="blue">
     <color rgba="0 0 0.8 1"/>

Commit message: update

File: orthrus_sim/orthrus_gazebo/models/orthrus/urdf/orthrus.urdf.xacro (robot description, xacro)
@@ -216,4 +216,16 @@
     <xacro:ros2_leg1_joint prefix="LB"/>
     <xacro:ros2_leg2_joint prefix="LB"/>
+    <sensor name="imu_sensor">
+      <state_interface name="orientation.x"/>
+      <state_interface name="orientation.y"/>
+      <state_interface name="orientation.z"/>
+      <state_interface name="angular_velocity.x"/>
+      <state_interface name="angular_velocity.y"/>
+      <state_interface name="angular_velocity.z"/>
+      <state_interface name="linear_acceleration.x"/>
+      <state_interface name="linear_acceleration.y"/>
+      <state_interface name="linear_acceleration.z"/>
+      <param name="frame_id">imu_link</param>
+    </sensor>
   </ros2_control>
   <gazebo>

File: orthrus_sim/orthrus_gazebo/models/orthrus/urdf/orthrus_for_gazebo.urdf.xacro (robot description, xacro)
@@ -3,5 +3,4 @@
   xmlns:xacro="http://ros.org/wiki/xacro">
   <xacro:property name="meshes_folder" value="file:///$(find orthrus_gazebo)/models/orthrus/meshes" />
-  <!--<xacro:property name="meshes_folder" value="/home/evence/code_file/ros2_ws/orthrus/src/orthrus_ros2_pack/orthrus_sim/orthrus_gazebo/models/orthrus/meshes" />-->
   <material name="blue">
     <color rgba="0 0 0.8 1"/>
@@ -32,8 +31,8 @@
     </inertial>
   </link>
-  <link name="dummy">
+  <link name="imu_link">
   </link>
-  <joint name="dummy_joint" type="fixed">
-    <parent link="dummy"/>
+  <joint name="imu_joint" type="fixed">
+    <parent link="imu_link"/>
     <child link="body"/>
   </joint>
@@ -222,4 +221,16 @@
     <xacro:ros2_leg1_joint prefix="LB"/>
     <xacro:ros2_leg2_joint prefix="LB"/>
+    <sensor name="imu_sensor">
+      <state_interface name="orientation.x"/>
+      <state_interface name="orientation.y"/>
+      <state_interface name="orientation.z"/>
+      <state_interface name="orientation.w"/>
+      <state_interface name="angular_velocity.x"/>
+      <state_interface name="angular_velocity.y"/>
+      <state_interface name="angular_velocity.z"/>
+      <state_interface name="linear_acceleration.x"/>
+      <state_interface name="linear_acceleration.y"/>
+      <state_interface name="linear_acceleration.z"/>
+    </sensor>
   </ros2_control>
   <gazebo>
