Commit message: update

File: orthrus_sim/orthrus_gazebo/models/orthrus/urdf/orthrus_for_gazebo.urdf.xacro (robot description, xacro)
@@ -62,5 +62,5 @@
       <parent link="body"/>
       <child link="hip_${prefix}"/>
-      <dynamics damping="0.1" friction="0.01"/>
+      <dynamics damping="0.4" friction="0.3"/>
       <limit effort="35.0" lower="-${pi/2}" upper="${pi/2}" velocity="${pi}"/>
       <xacro:if value="${prefix == 'LF'}">
@@ -106,5 +106,5 @@
       <parent link="hip_${prefix}"/>
       <child link="leg1_${prefix}"/>
-      <dynamics damping="0.1" friction="0.01"/>
+      <dynamics damping="0.4" friction="0.3"/>
       <limit effort="35.0" lower="-${pi*2/3}" upper="${pi*2/3}" velocity="${pi}"/>
       <xacro:if value="${prefix == 'LF'}">
@@ -150,5 +150,5 @@
       <parent link="leg1_${prefix}"/>
       <child link="leg2_${prefix}"/>
-      <dynamics damping="0.1" friction="0.01"/>
+      <dynamics damping="0.4" friction="0.3"/>
       <xacro:if value="${prefix == 'LF'}">
         <origin xyz="0.035 -0.18 0" rpy="${pi*2/3} 0 0" />

Commit message: update

File: orthrus_sim/orthrus_gazebo/models/orthrus/urdf/orthrus_for_gazebo.urdf.xacro (robot description, xacro)
@@ -34,6 +34,6 @@
   </link>
   <joint name="imu_joint" type="fixed">
-    <parent link="imu_link"/>
-    <child link="body"/>
+    <parent link="body"/>
+    <child link="imu_link"/>
   </joint>
   <xacro:macro name="hip" params="prefix">
