Commit message: update

File: orthrus_sim/orthrus_ign/models/orthrus/urdf/orthrus.urdf (robot description, URDF)
Before this commit: robot orthrus, 13 links, 12 joints
Links:
- link body: geometry visual mesh filename=file:////home/evence/code_file/ros2_ws/orthrus/install/orth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
- link hip_LB: geometry visual mesh filename=file:////home/evence/code_file/ros2_ws/orthrus/install/orth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
- link hip_LF: geometry visual mesh filename=file:////home/evence/code_file/ros2_ws/orthrus/install/orth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
- link hip_RB: geometry visual mesh filename=file:////home/evence/code_file/ros2_ws/orthrus/install/orth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
- link hip_RF: geometry visual mesh filename=file:////home/evence/code_file/ros2_ws/orthrus/install/orth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
- link leg1_LB: geometry visual mesh filename=file:////home/evence/code_file/ros2_ws/orthrus/install/orth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
- link leg1_LF: geometry visual mesh filename=file:////home/evence/code_file/ros2_ws/orthrus/install/orth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
- link leg1_RB: geometry visual mesh filename=file:////home/evence/code_file/ros2_ws/orthrus/install/orth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
- link leg1_RF: geometry visual mesh filename=file:////home/evence/code_file/ros2_ws/orthrus/install/orth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
- link leg2_LB: geometry visual mesh filename=file:////home/evence/code_file/ros2_ws/orthrus/install/orth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
- link leg2_LF: geometry visual mesh filename=file:////home/evence/code_file/ros2_ws/orthrus/install/orth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
- link leg2_RB: geometry visual mesh filename=file:////home/evence/code_file/ros2_ws/orthrus/install/orth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
- link leg2_RF: geometry visual mesh filename=file:////home/evence/code_file/ros2_ws/orthrus/install/orth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
