Commit message: update

File: orthrus_interfaces/models/a1/urdf/robot.urdf (robot description, URDF)
Before this commit: robot robot, 18 links, 17 joints
Links:
- link LF_calf: geometry collision box size=0.2 0.016 0.016; visual mesh filename=/home/orthrus/orthrus/install/orthrus_interfaces/share/orth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 scale=1 1 1
- link LF_hip: geometry collision cylinder length=0.04 radius=0.046; visual mesh filename=/home/orthrus/orthrus/install/orthrus_interfaces/share/orth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 scale=1 1 1
- link LF_thigh: geometry collision box size=0.2 0.03 0.034; collision cylinder length=0.04 radius=0.041
- link LH_calf: geometry collision box size=0.2 0.016 0.016; visual mesh filename=/home/orthrus/orthrus/install/orthrus_interfaces/share/orth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 scale=1 1 1
- link LH_hip: geometry collision cylinder length=0.04 radius=0.046; visual mesh filename=/home/orthrus/orthrus/install/orthrus_interfaces/share/orth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 scale=1 1 1
- link LH_thigh: geometry collision box size=0.2 0.03 0.034; collision cylinder length=0.04 radius=0.041
- link RF_calf: geometry collision box size=0.2 0.016 0.016; visual mesh filename=/home/orthrus/orthrus/install/orthrus_interfaces/share/orth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 scale=1 1 1
- link RF_hip: geometry collision cylinder length=0.04 radius=0.046; visual mesh filename=/home/orthrus/orthrus/install/orthrus_interfaces/share/orth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 scale=1 1 1
- link RF_thigh: geometry collision box size=0.2 0.03 0.034; collision cylinder length=0.04 radius=0.041
- link RH_calf: geometry collision box size=0.2 0.016 0.016; visual mesh filename=/home/orthrus/orthrus/install/orthrus_interfaces/share/orth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 scale=1 1 1
- link RH_hip: geometry collision cylinder length=0.04 radius=0.046; visual mesh filename=/home/orthrus/orthrus/install/orthrus_interfaces/share/orth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 scale=1 1 1
- link RH_thigh: geometry collision box size=0.2 0.03 0.034; collision cylinder length=0.04 radius=0.041
- link base: geometry collision box size=0.267 0.194 0.114; visual mesh filename=/home/orthrus/orthrus/install/orthrus_interfaces/share/orth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 scale=1 1 1

File: orthrus_interfaces/models/orthrus/urdf/orthrus.urdf (robot description, URDF)
Before this commit: robot orthrus, 13 links, 12 joints
Links:
- link LF_HAA_link: geometry collision mesh filename=file:////home/orthrus/orthrus/install/orthrus_interfaces/sh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; visual mesh filename=file:////home/orthrus/orthrus/install/orthrus_interfaces/sh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
- link LF_HFE_link: geometry collision mesh filename=file:////home/orthrus/orthrus/install/orthrus_interfaces/sh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; visual mesh filename=file:////home/orthrus/orthrus/install/orthrus_interfaces/sh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
- link LF_KFE_link: geometry collision mesh filename=file:////home/orthrus/orthrus/install/orthrus_interfaces/sh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; visual mesh filename=file:////home/orthrus/orthrus/install/orthrus_interfaces/sh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
- link LH_HAA_link: geometry collision mesh filename=file:////home/orthrus/orthrus/install/orthrus_interfaces/sh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; visual mesh filename=file:////home/orthrus/orthrus/install/orthrus_interfaces/sh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
- link LH_HFE_link: geometry collision mesh filename=file:////home/orthrus/orthrus/install/orthrus_interfaces/sh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; visual mesh filename=file:////home/orthrus/orthrus/install/orthrus_interfaces/sh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
- link LH_KFE_link: geometry collision mesh filename=file:////home/orthrus/orthrus/install/orthrus_interfaces/sh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; visual mesh filename=file:////home/orthrus/orthrus/install/orthrus_interfaces/sh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
- link RF_HAA_link: geometry collision mesh filename=file:////home/orthrus/orthrus/install/orthrus_interfaces/sh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; visual mesh filename=file:////home/orthrus/orthrus/install/orthrus_interfaces/sh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
- link RF_HFE_link: geometry collision mesh filename=file:////home/orthrus/orthrus/install/orthrus_interfaces/sh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; visual mesh filename=file:////home/orthrus/orthrus/install/orthrus_interfaces/sh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
- link RF_KFE_link: geometry collision mesh filename=file:////home/orthrus/orthrus/install/orthrus_interfaces/sh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; visual mesh filename=file:////home/orthrus/orthrus/install/orthrus_interfaces/sh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
- link RH_HAA_link: geometry collision mesh filename=file:////home/orthrus/orthrus/install/orthrus_interfaces/sh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; visual mesh filename=file:////home/orthrus/orthrus/install/orthrus_interfaces/sh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
- link RH_HFE_link: geometry collision mesh filename=file:////home/orthrus/orthrus/install/orthrus_interfaces/sh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; visual mesh filename=file:////home/orthrus/orthrus/install/orthrus_interfaces/sh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
- link RH_KFE_link: geometry collision mesh filename=file:////home/orthrus/orthrus/install/orthrus_interfaces/sh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; visual mesh filename=file:////home/orthrus/orthrus/install/orthrus_interfaces/sh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
- link base: geometry collision mesh filename=file:////home/orthrus/orthrus/install/orthrus_interfaces/sh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; visual mesh filename=file:////home/orthrus/orthrus/install/orthrus_interfaces/sh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

File: orthrus_interfaces/models/orthrus/urdf/orthrus.urdf.xacro (robot description, xacro)
@@ -53,5 +53,5 @@
   <gazebo>
     <plugin filename="libgazebo_ros2_control.so" name="gazebo_ros2_control">
-      <parameters>/home/evence/code_file/ros2_ws/orthrus/src/orthrus_ros2_pack/orthrus_sim/orthrus_gazebo/config/orthrus.yaml</parameters>
+      <parameters>/home/orthrus/orthrus/src/orthrus_ros2_pack/orthrus_sim/orthrus_gazebo/config/orthrus.yaml</parameters>
     </plugin>
   </gazebo>

Commit message: update

File: orthrus_interfaces/models/a1/urdf/robot.urdf (robot description, URDF)
Before this commit: robot robot, 18 links, 17 joints
Links:
- link LF_calf: geometry collision box size=0.2 0.016 0.016; visual mesh filename=/home/evence/code_file/ros2_ws/orthrus/install/orthrus_inte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 scale=1 1 1
- link LF_hip: geometry collision cylinder length=0.04 radius=0.046; visual mesh filename=/home/evence/code_file/ros2_ws/orthrus/install/orthrus_inte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 scale=1 1 1
- link LF_thigh: geometry collision box size=0.2 0.03 0.034; collision cylinder length=0.04 radius=0.041
- link LH_calf: geometry collision box size=0.2 0.016 0.016; visual mesh filename=/home/evence/code_file/ros2_ws/orthrus/install/orthrus_inte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 scale=1 1 1
- link LH_hip: geometry collision cylinder length=0.04 radius=0.046; visual mesh filename=/home/evence/code_file/ros2_ws/orthrus/install/orthrus_inte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 scale=1 1 1
- link LH_thigh: geometry collision box size=0.2 0.03 0.034; collision cylinder length=0.04 radius=0.041
- link RF_calf: geometry collision box size=0.2 0.016 0.016; visual mesh filename=/home/evence/code_file/ros2_ws/orthrus/install/orthrus_inte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 scale=1 1 1
- link RF_hip: geometry collision cylinder length=0.04 radius=0.046; visual mesh filename=/home/evence/code_file/ros2_ws/orthrus/install/orthrus_inte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 scale=1 1 1
- link RF_thigh: geometry collision box size=0.2 0.03 0.034; collision cylinder length=0.04 radius=0.041
- link RH_calf: geometry collision box size=0.2 0.016 0.016; visual mesh filename=/home/evence/code_file/ros2_ws/orthrus/install/orthrus_inte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 scale=1 1 1
- link RH_hip: geometry collision cylinder length=0.04 radius=0.046; visual mesh filename=/home/evence/code_file/ros2_ws/orthrus/install/orthrus_inte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 scale=1 1 1
- link RH_thigh: geometry collision box size=0.2 0.03 0.034; collision cylinder length=0.04 radius=0.041
- link base: geometry collision box size=0.267 0.194 0.114; visual mesh filename=/home/evence/code_file/ros2_ws/orthrus/install/orthrus_inte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 scale=1 1 1

File: orthrus_interfaces/models/orthrus/urdf/orthrus.urdf (robot description, URDF)
Before this commit: robot orthrus, 13 links, 12 joints
Links:
- added link LF_FOOT_link
- added link LH_FOOT_link
- added link RF_FOOT_link
- added link RH_FOOT_link
- link LF_HAA_link: geometry collision mesh filename=file:////home/evence/code_file/ros2_ws/orthrus/install/orth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; visual mesh filename=file:////home/evence/code_file/ros2_ws/orthrus/install/orth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
- link LF_HFE_link: geometry collision mesh filename=file:////home/evence/code_file/ros2_ws/orthrus/install/orth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; visual mesh filename=file:////home/evence/code_file/ros2_ws/orthrus/install/orth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
- link LF_KFE_link: geometry collision mesh filename=file:////home/evence/code_file/ros2_ws/orthrus/install/orth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; visual mesh filename=file:////home/evence/code_file/ros2_ws/orthrus/install/orth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
- link LH_HAA_link: geometry collision mesh filename=file:////home/evence/code_file/ros2_ws/orthrus/install/orth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; visual mesh filename=file:////home/evence/code_file/ros2_ws/orthrus/install/orth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
- link LH_HFE_link: geometry collision mesh filename=file:////home/evence/code_file/ros2_ws/orthrus/install/orth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; visual mesh filename=file:////home/evence/code_file/ros2_ws/orthrus/install/orth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
- link LH_KFE_link: geometry collision mesh filename=file:////home/evence/code_file/ros2_ws/orthrus/install/orth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; visual mesh filename=file:////home/evence/code_file/ros2_ws/orthrus/install/orth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
- link RF_HAA_link: geometry collision mesh filename=file:////home/evence/code_file/ros2_ws/orthrus/install/orth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; visual mesh filename=file:////home/evence/code_file/ros2_ws/orthrus/install/orth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
- link RF_HFE_link: geometry collision mesh filename=file:////home/evence/code_file/ros2_ws/orthrus/install/orth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; visual mesh filename=file:////home/evence/code_file/ros2_ws/orthrus/install/orth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
- link RF_KFE_link: geometry collision mesh filename=file:////home/evence/code_file/ros2_ws/orthrus/install/orth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; visual mesh filename=file:////home/evence/code_file/ros2_ws/orthrus/install/orth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
- link RH_HAA_link: geometry collision mesh filename=file:////home/evence/code_file/ros2_ws/orthrus/install/orth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; visual mesh filename=file:////home/evence/code_file/ros2_ws/orthrus/install/orth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
- link RH_HFE_link: geometry collision mesh filename=file:////home/evence/code_file/ros2_ws/orthrus/install/orth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; visual mesh filename=file:////home/evence/code_file/ros2_ws/orthrus/install/orth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
- link RH_KFE_link: geometry collision mesh filename=file:////home/evence/code_file/ros2_ws/orthrus/install/orth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; visual mesh filename=file:////home/evence/code_file/ros2_ws/orthrus/install/orth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
- link base: geometry collision mesh filename=file:////home/evence/code_file/ros2_ws/orthrus/install/orth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; visual mesh filename=file:////home/evence/code_file/ros2_ws/orthrus/install/orth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
Joints:
- added joint LF_FOOT: type fixed, parent LF_KFE_link, child LF_FOOT_link, origin xyz=0.0 0.0 -0.2 rpy=0 0 0, axis 1 0 0
- added joint LH_FOOT: type fixed, parent LH_KFE_link, child LH_FOOT_link, origin xyz=0.0 0.0 -0.2 rpy=0 0 0, axis 1 0 0
- added joint RF_FOOT: type fixed, parent RF_KFE_link, child RF_FOOT_link, origin xyz=0.0 0.0 -0.2 rpy=0 0 0, axis 1 0 0
- added joint RH_FOOT: type fixed, parent RH_KFE_link, child RH_FOOT_link, origin xyz=0.0 0.0 -0.2 rpy=0 0 0, axis 1 0 0

File: orthrus_interfaces/models/orthrus/urdf/orthrus.urdf.xacro (robot description, xacro)
@@ -53,5 +53,5 @@
   <gazebo>
     <plugin filename="libgazebo_ros2_control.so" name="gazebo_ros2_control">
-      <parameters>/home/orthrus/orthrus/src/orthrus_ros2_pack/orthrus_sim/orthrus_gazebo/config/orthrus.yaml</parameters>
+      <parameters>/home/evence/code_file/ros2_ws/orthrus/src/orthrus_ros2_pack/orthrus_sim/orthrus_gazebo/config/orthrus.yaml</parameters>
     </plugin>
   </gazebo>

File: orthrus_interfaces/models/orthrus/urdf/orthrus_base.xacro (robot description, xacro)
@@ -44,6 +44,7 @@
       </collision>
       <inertial>
+        <origin xyz="0.01493 0.00159 0.00" rpy="0 0 0" />
         <mass value="0.7"/>
-        <inertia ixx="0.0904981" ixy="0" ixz="-0.0000480" iyy=" 0.0917319" iyz="0" izz="0.0857923" />
+        <inertia ixx="-0.084" ixy="0.0" ixz="0.996" iyy="-1.0" iyz="0.0" izz="0.084" />
       </inertial>
     </link>
@@ -84,4 +85,5 @@
       </collision>
       <inertial>
+        <origin xyz="0.02764 -0.02513 0.00" rpy="0 0 0" />
         <mass value="1"/>
         <inertia ixx="0.4329464" ixy="-0.0830239" ixz=" -0.0000001" iyy="0.1503071" iyz="0.0000001" izz="0.4817994" />
@@ -124,4 +126,5 @@
       </collision>
       <inertial>
+        <origin xyz="0.00 0.00 -0.12564" rpy="0 0 0" />
         <mass value="0.2"/>
         <inertia ixx="0.4201680" ixy="0" ixz="0" iyy="0.4196489" iyz="0" izz="0.0031965" />
@@ -149,4 +152,14 @@
         <limit effort="35.0" lower="-${pi*1/12}" upper="${pi*2/3}" velocity="${pi}"/>
       </xacro:if>
+    </joint>
+  </xacro:macro>
+  <xacro:macro name="FOOT" params="prefix">
+    <link name="${prefix}_FOOT_link">
+    </link>
+    <joint name="${prefix}_FOOT" type="fixed">
+      <axis xyz="1 0 0"/>
+      <parent link="${prefix}_KFE_link"/>
+      <child link="${prefix}_FOOT_link"/>
+      <origin xyz="0.0 0.0 -0.2" rpy="0 0 0" />
     </joint>
   </xacro:macro>
@@ -184,3 +197,7 @@
     </joint>
   </xacro:macro>
+  <xacro:macro name="ros2_FOOT_joint" params="prefix">
+    <joint name="${prefix}_FOOT">
+    </joint>
+  </xacro:macro>
 </robot>
