Commit message: update

File: orthrus_interfaces/models/orthrus/urdf/orthrus.urdf.xacro (robot description, xacro)
@@ -14,10 +14,4 @@
   <xacro:leg2 prefix="LB"/>
   <xacro:leg2 prefix="RB"/>
-  <link name="horizontal">
-  </link>
-  <joint name="horizontal_joint" type="floating">
-    <parent link="body"/>
-    <child link="horizontal"/>
-  </joint>
   <ros2_control name="GazeboSystem" type="system">
     <hardware>

Commit message: update

File: orthrus_interfaces/models/orthrus/urdf/orthrus.urdf.xacro (robot description, xacro)
@@ -2,5 +2,5 @@
 <robot name="orthrus"
   xmlns:xacro="http://ros.org/wiki/xacro">
-  <xacro:property name="meshes_folder" value="file:///$(find orthrus_gazebo)/models/orthrus/meshes" />
+  <xacro:property name="meshes_folder" value="file:///$(find orthrus_interfaces)/models/orthrus/meshes" />
   <xacro:include filename="orthrus_base.xacro"/>
   <xacro:HAA prefix="RF"/>

File: orthrus_interfaces/models/orthrus/urdf/orthrus_base.xacro (robot description, xacro)
@@ -29,5 +29,5 @@
   </link>
   <xacro:macro name="HAA" params="prefix">
-    <link name="${prefix}_HAA">
+    <link name="${prefix}_HAA_link">
       <visual>
         <origin xyz="-0.02 -0.05 -0.05" rpy="0 0 0" />
@@ -51,5 +51,5 @@
       <axis xyz="0 0 1"/>
       <parent link="base"/>
-      <child link="${prefix}_HAA"/>
+      <child link="${prefix}_HAA_link"/>
       <dynamics damping="0.4" friction="0.3"/>
       <limit effort="35.0" lower="-${pi/2}" upper="${pi/2}" velocity="${pi}"/>
@@ -69,5 +69,5 @@
   </xacro:macro>
   <xacro:macro name="HFE" params="prefix">
-    <link name="${prefix}_HFE">
+    <link name="${prefix}_HFE_link">
       <visual>
         <origin xyz="0 -0.2 -0.05" rpy="0 0 0" />
@@ -90,6 +90,6 @@
     <joint name="${prefix}_HFE" type="revolute">
       <axis xyz="1 0 0"/>
-      <parent link="${prefix}_HAA"/>
-      <child link="${prefix}_HFE"/>
+      <parent link="${prefix}_HAA_link"/>
+      <child link="${prefix}_HFE_link"/>
       <dynamics damping="0.4" friction="0.3"/>
       <limit effort="35.0" lower="-${pi*2/3}" upper="${pi*2/3}" velocity="${pi}"/>
@@ -109,5 +109,5 @@
   </xacro:macro>
   <xacro:macro name="KFE" params="prefix">
-    <link name="${prefix}_KFE">
+    <link name="${prefix}_KFE_link">
       <visual>
         <origin xyz="-0.025 -0.025 -0.225" rpy="0 0 0" />
@@ -130,6 +130,6 @@
     <joint name="${prefix}_KFE" type="revolute">
       <axis xyz="1 0 0"/>
-      <parent link="${prefix}_HFE"/>
-      <child link="${prefix}_KFE"/>
+      <parent link="${prefix}_HFE_link"/>
+      <child link="${prefix}_KFE_link"/>
       <dynamics damping="0.4" friction="0.3"/>
       <xacro:if value="${prefix == 'LF'}">
@@ -152,5 +152,5 @@
   </xacro:macro>
   <xacro:macro name="ros2_HAA_joint" params="prefix">
-    <joint name="HAA_${prefix}_joint">
+    <joint name="${prefix}_HAA">
       <command_interface name="effort">
         <param name="min">-35</param>
@@ -163,5 +163,5 @@
   </xacro:macro>
   <xacro:macro name="ros2_HFE_joint" params="prefix">
-    <joint name="HFE_${prefix}_joint">
+    <joint name="${prefix}_HFE">
       <command_interface name="effort">
         <param name="min">-35</param>
@@ -174,5 +174,5 @@
   </xacro:macro>
   <xacro:macro name="ros2_KFE_joint" params="prefix">
-    <joint name="KFE_${prefix}_joint">
+    <joint name="${prefix}_KFE">
       <command_interface name="effort">
         <param name="min">-35</param>

File: orthrus_interfaces/models/orthrus/urdf/orthrus_for_gazebo.urdf.xacro (robot description, xacro)
@@ -2,5 +2,5 @@
 <robot name="orthrus"
   xmlns:xacro="http://ros.org/wiki/xacro">
-  <xacro:property name="meshes_folder" value="file:///$(find orthrus_gazebo)/models/orthrus/meshes" />
+  <xacro:property name="meshes_folder" value="file:///$(find orthrus_interfaces)/models/orthrus/meshes" />
   <xacro:include filename="orthrus_base.xacro"/>
   <xacro:HAA prefix="RF"/>
@@ -16,5 +16,5 @@
   <xacro:KFE prefix="LH"/>
   <xacro:KFE prefix="RH"/>
-  <gazebo reference="body">
+  <gazebo reference="base">
     <sensor name="imu_sensor" type="imu">
       <always_on>1</always_on>

Commit message: update

File: orthrus_interfaces/models/orthrus/urdf/orthrus.urdf.xacro (robot description, xacro)
@@ -3,4 +3,5 @@
   xmlns:xacro="http://ros.org/wiki/xacro">
   <xacro:property name="meshes_folder" value="file:///$(find orthrus_interfaces)/models/orthrus/meshes" />
+  <xacro:property name="orthrus_config_path" value="$(find orthrus_gazebo)/config/orthrus.yaml" />
   <xacro:include filename="orthrus_base.xacro"/>
   <xacro:HAA prefix="LF"/>
@@ -61,5 +62,5 @@
   <gazebo>
     <plugin filename="libgazebo_ros2_control.so" name="gazebo_ros2_control">
-      <parameters>/home/orthrus/orthrus/src/orthrus_ros2_pack/orthrus_sim/orthrus_gazebo/config/orthrus.yaml</parameters>
+      <parameters><xacro:property name="orthrus_config_path" value="$(find orthrus_gazebo)/config/orthrus.yaml" /></parameters>
     </plugin>
   </gazebo>

Commit message: update

File: orthrus_interfaces/models/orthrus/urdf/orthrus.urdf.xacro (robot description, xacro)
@@ -3,5 +3,5 @@
   xmlns:xacro="http://ros.org/wiki/xacro">
   <xacro:property name="meshes_folder" value="file:///$(find orthrus_interfaces)/models/orthrus/meshes" />
-  <xacro:property name="orthrus_config_path" value="$(find orthrus_gazebo)/config/orthrus.yaml" />
+  <xacro:property name="orthrus_config_path" value="file:///$(find orthrus_gazebo)/config/orthrus.yaml" />
   <xacro:include filename="orthrus_base.xacro"/>
   <xacro:HAA prefix="LF"/>
@@ -62,5 +62,5 @@
   <gazebo>
     <plugin filename="libgazebo_ros2_control.so" name="gazebo_ros2_control">
-      <parameters><xacro:property name="orthrus_config_path" value="$(find orthrus_gazebo)/config/orthrus.yaml" /></parameters>
+      <parameters>$(find orthrus_gazebo)/config/orthrus.yaml</parameters>
     </plugin>
   </gazebo>
