Commit message: update

File: orthrus_interfaces/models/orthrus/urdf/orthrus_base.xacro (robot description, xacro)
@@ -11,5 +11,5 @@
   <link name="base">
     <visual>
-      <origin xyz="-0.10 0.1385 -0.05" rpy="${pi/2} 0 0" />
+      <origin xyz="-0.1385 -0.10 -0.05" rpy="${pi/2} 0 ${pi/2}" />
       <geometry>
         <mesh filename="${meshes_folder}/body.STL"/>
@@ -18,5 +18,5 @@
     </visual>
     <collision>
-      <origin xyz="-0.10 0.1385 -0.05" rpy="${pi/2} 0 0" />
+      <origin xyz="-0.1385 -0.10 -0.05" rpy="${pi/2} 0 ${pi/2}" />
       <geometry>
         <mesh filename="${meshes_folder}/body.STL"/>
@@ -25,5 +25,5 @@
     <inertial>
       <mass value="7"/>
-      <inertia ixx="4.9950395" ixy="0" ixz="0" iyy="2.4616377" iyz="0" izz="6.4183150" />
+      <inertia ixx="2.4616377" ixy="0" ixz="0" iyy="4.9950395" iyz="0" izz="6.4183150" />
     </inertial>
   </link>
@@ -55,14 +55,14 @@
       <limit effort="35.0" lower="-${pi/2}" upper="${pi/2}" velocity="${pi}"/>
       <xacro:if value="${prefix == 'LF'}">
-        <origin xyz="-0.05 0.20 0" rpy="${pi/2} ${pi} 0" />
+        <origin xyz="0.20 0.05 0" rpy="${pi/2} ${pi} ${-pi/2}" />
       </xacro:if>
       <xacro:if value="${prefix == 'LH'}">
-        <origin xyz="-0.05 -0.20 0" rpy="-${pi/2} ${pi} 0" />
+        <origin xyz="-0.20 0.05 0" rpy="-${pi/2} ${pi} ${-pi/2}" />
       </xacro:if>
       <xacro:if value="${prefix == 'RH'}">
-        <origin xyz="0.05 -0.20 0" rpy="${pi/2} ${pi} ${pi}" />
+        <origin xyz="-0.20 -0.05 0" rpy="${pi/2} ${pi} ${pi/2}" />
       </xacro:if>
       <xacro:if value="${prefix == 'RF'}">
-        <origin xyz="0.05 0.20 0" rpy="-${pi/2} ${pi} ${pi}" />
+        <origin xyz="0.20 -0.05 0" rpy="-${pi/2} ${pi} ${pi/2}" />
       </xacro:if>
     </joint>

Commit message: update

File: orthrus_interfaces/models/orthrus/urdf/orthrus_base.xacro (robot description, xacro)
@@ -202,3 +202,45 @@
     </joint>
   </xacro:macro>
+  <xacro:macro name="orthrus_ros2_control" params="prefix">
+    <ros2_control name="GazeboSystem" type="system">
+      <xacro:if value="${prefix == 'gazebo'}">
+        <hardware>
+          <plugin>gazebo_ros2_control/GazeboSystem</plugin>
+        </hardware>
+      </xacro:if>
+      <xacro:if value="${prefix == 'real'}">
+        <hardware>
+          <plugin>"orthrus_control/OrthrusSystemHardware</plugin>
+        </hardware>
+      </xacro:if>
+      <xacro:ros2_HAA_joint prefix="RF"/>
+      <xacro:ros2_HFE_joint prefix="RF"/>
+      <xacro:ros2_KFE_joint prefix="RF"/>
+      <xacro:ros2_FOOT_joint prefix="RF"/>
+      <xacro:ros2_HAA_joint prefix="LF"/>
+      <xacro:ros2_HFE_joint prefix="LF"/>
+      <xacro:ros2_KFE_joint prefix="LF"/>
+      <xacro:ros2_FOOT_joint prefix="LF"/>
+      <xacro:ros2_HAA_joint prefix="RH"/>
+      <xacro:ros2_HFE_joint prefix="RH"/>
+      <xacro:ros2_KFE_joint prefix="RH"/>
+      <xacro:ros2_FOOT_joint prefix="RH"/>
+      <xacro:ros2_HAA_joint prefix="LH"/>
+      <xacro:ros2_HFE_joint prefix="LH"/>
+      <xacro:ros2_KFE_joint prefix="LH"/>
+      <xacro:ros2_FOOT_joint prefix="LH"/>
+      <sensor name="imu_sensor">
+        <state_interface name="orientation.x"/>
+        <state_interface name="orientation.y"/>
+        <state_interface name="orientation.z"/>
+        <state_interface name="orientation.w"/>
+        <state_interface name="angular_velocity.x"/>
+        <state_interface name="angular_velocity.y"/>
+        <state_interface name="angular_velocity.z"/>
+        <state_interface name="linear_acceleration.x"/>
+        <state_interface name="linear_acceleration.y"/>
+        <state_interface name="linear_acceleration.z"/>
+      </sensor>
+    </ros2_control>
+  </xacro:macro>
 </robot>

File: orthrus_interfaces/models/orthrus/urdf/orthrus_gazebo.urdf.xacro (robot description, xacro)
@@ -1,5 +1,3 @@
-<?xml version="1.0"?>
-<robot name="orthrus"
-  xmlns:xacro="http://ros.org/wiki/xacro">
+<robot name="orthrus" xmlns:xacro="http://ros.org/wiki/xacro">
   <xacro:property name="meshes_folder" value="file:///$(find orthrus_interfaces)/models/orthrus/meshes" />
   <xacro:property name="orthrus_config_path" value="file:///$(find orthrus_gazebo)/config/orthrus.yaml" />
@@ -21,4 +19,5 @@
   <xacro:KFE prefix="RH"/>
   <xacro:FOOT prefix="RH"/>
+  <xacro:orthrus_ros2_control prefix="gazebo"/>
   <gazebo reference="base">
     <sensor name="imu_sensor" type="imu">

File: orthrus_interfaces/models/orthrus/urdf/orthrus_real.urdf.xacro (robot description, xacro)
@@ -21,4 +21,5 @@
   <xacro:KFE prefix="RH"/>
   <xacro:FOOT prefix="RH"/>
+  <xacro:orthrus_ros2_control prefix="real"/>
   <gazebo reference="base">
     <sensor name="imu_sensor" type="imu">

Commit message: update

File: orthrus_interfaces/models/orthrus/urdf/orthrus_base.xacro (robot description, xacro)
@@ -198,10 +198,6 @@
     </joint>
   </xacro:macro>
-  <xacro:macro name="ros2_FOOT_joint" params="prefix">
-    <joint name="${prefix}_FOOT">
-    </joint>
-  </xacro:macro>
-  <xacro:macro name="orthrus_ros2_control" params="prefix">
-    <ros2_control name="GazeboSystem" type="system">
+  <xacro:macro name="orthrus_ros2_control" params="prefix name">
+    <ros2_control name="${name}" type="system">
       <xacro:if value="${prefix == 'gazebo'}">
         <hardware>
@@ -211,5 +207,5 @@
       <xacro:if value="${prefix == 'real'}">
         <hardware>
-          <plugin>"orthrus_control/OrthrusSystemHardware</plugin>
+          <plugin>orthrus_control/OrthrusSystemHardware</plugin>
         </hardware>
       </xacro:if>
@@ -217,17 +213,13 @@
       <xacro:ros2_HFE_joint prefix="RF"/>
       <xacro:ros2_KFE_joint prefix="RF"/>
-      <xacro:ros2_FOOT_joint prefix="RF"/>
       <xacro:ros2_HAA_joint prefix="LF"/>
       <xacro:ros2_HFE_joint prefix="LF"/>
       <xacro:ros2_KFE_joint prefix="LF"/>
-      <xacro:ros2_FOOT_joint prefix="LF"/>
       <xacro:ros2_HAA_joint prefix="RH"/>
       <xacro:ros2_HFE_joint prefix="RH"/>
       <xacro:ros2_KFE_joint prefix="RH"/>
-      <xacro:ros2_FOOT_joint prefix="RH"/>
       <xacro:ros2_HAA_joint prefix="LH"/>
       <xacro:ros2_HFE_joint prefix="LH"/>
       <xacro:ros2_KFE_joint prefix="LH"/>
-      <xacro:ros2_FOOT_joint prefix="LH"/>
       <sensor name="imu_sensor">
         <state_interface name="orientation.x"/>

File: orthrus_interfaces/models/orthrus/urdf/orthrus_gazebo.urdf.xacro (robot description, xacro)
@@ -19,5 +19,5 @@
   <xacro:KFE prefix="RH"/>
   <xacro:FOOT prefix="RH"/>
-  <xacro:orthrus_ros2_control prefix="gazebo"/>
+  <xacro:orthrus_ros2_control prefix="gazebo" name="GazeboSystem"/>
   <gazebo reference="base">
     <sensor name="imu_sensor" type="imu">

File: orthrus_interfaces/models/orthrus/urdf/orthrus_real.urdf.xacro (robot description, xacro)
@@ -21,15 +21,4 @@
   <xacro:KFE prefix="RH"/>
   <xacro:FOOT prefix="RH"/>
-  <xacro:orthrus_ros2_control prefix="real"/>
-  <gazebo reference="base">
-    <sensor name="imu_sensor" type="imu">
-      <always_on>1</always_on>
-      <update_rate>1000</update_rate>
-    </sensor>
-  </gazebo>
-  <gazebo>
-    <plugin filename="libgazebo_ros2_control.so" name="gazebo_ros2_control">
-      <parameters>$(find orthrus_gazebo)/config/orthrus.yaml</parameters>
-    </plugin>
-  </gazebo>
+  <xacro:orthrus_ros2_control prefix="real" name="OrthrusSystemHardware"/>
 </robot>

Commit message: update

File: orthrus_interfaces/models/orthrus/urdf/orthrus_base.xacro (robot description, xacro)
@@ -25,6 +25,7 @@
     </collision>
     <inertial>
-      <mass value="7"/>
-      <inertia ixx="2.4616377" ixy="0" ixz="0" iyy="4.9950395" iyz="0" izz="6.4183150" />
+      <origin xyz="-0.010977 0.000003 -0.000477" rpy="0 0 0" />
+      <mass value="4.429"/>
+      <inertia ixx="1.4923275" ixy="-0.0034837" ixz=" -0.0020438" iyy="5.0690680" iyz="0.0209222" izz="5.7629196" />
     </inertial>
   </link>

Commit message: update

File: orthrus_interfaces/models/orthrus/urdf/orthrus_base.xacro (robot description, xacro)
@@ -27,5 +27,5 @@
       <origin xyz="-0.010977 0.000003 -0.000477" rpy="0 0 0" />
       <mass value="4.429"/>
-      <inertia ixx="1.4923275" ixy="-0.0034837" ixz=" -0.0020438" iyy="5.0690680" iyz="0.0209222" izz="5.7629196" />
+      <inertia ixx="0.014923275" ixy="-0.000034837" ixz=" -0.000020438" iyy="0.050690680" iyz="0.000209222" izz="0.057629196" />
     </inertial>
   </link>
@@ -46,7 +46,7 @@
       </collision>
       <inertial>
-        <origin xyz="0.01493 0.00159 0.00" rpy="0 0 0" />
-        <mass value="0.7"/>
-        <inertia ixx="-0.084" ixy="0.0" ixz="0.996" iyy="-1.0" iyz="0.0" izz="0.084" />
+        <origin xyz="0.003391 0.000355 0.001734" rpy="0 0 0" />
+        <mass value="0.67"/>
+        <inertia ixx="-0.000849931" ixy="-0.000005571" ixz="0.000007520" iyy="0.000608499" iyz="-0.000003845" izz="0.000546025" />
       </inertial>
     </link>
@@ -87,7 +87,24 @@
       </collision>
       <inertial>
-        <origin xyz="0.02764 -0.02513 0.00" rpy="0 0 0" />
-        <mass value="1"/>
-        <inertia ixx="0.4329464" ixy="-0.0830239" ixz=" -0.0000001" iyy="0.1503071" iyz="0.0000001" izz="0.4817994" />
+        <xacro:if value="${prefix == 'LF'}">
+          <origin xyz="0.013465 -0.021755 -0.000094" rpy="0 0 0" />
+          <mass value="0.928"/>
+          <inertia ixx="0.003597820" ixy="-0.000526099" ixz="-0.000000377" iyy="0.001042179" iyz="0.000060684" izz="0.003628939" />
+        </xacro:if>
+        <xacro:if value="${prefix == 'LH'}">
+          <origin xyz="0.013465 -0.021755 -0.000094" rpy="0 0 0" />
+          <mass value="0.928"/>
+          <inertia ixx="0.003597820" ixy="-0.000526099" ixz="-0.000000377" iyy="0.001042179" iyz="0.000060684" izz="0.003628939" />
+        </xacro:if>
+        <xacro:if value="${prefix == 'RH'}">
+          <origin xyz="0.013465 -0.021755 0.000094" rpy="0 0 0" />
+          <mass value="0.928"/>
+          <inertia ixx="0.003597820" ixy="-0.000526099" ixz="-0.000000377" iyy="0.001042179" iyz="0.000060684" izz="0.003628939" />
+        </xacro:if>
+        <xacro:if value="${prefix == 'RF'}">
+          <origin xyz="0.013465 -0.021755 0.000094" rpy="0 0 0" />
+          <mass value="0.928"/>
+          <inertia ixx="0.003597820" ixy="-0.000526099" ixz="-0.000000377" iyy="0.001042179" iyz="0.000060684" izz="0.003628939" />
+        </xacro:if>
       </inertial>
     </link>
@@ -128,7 +145,24 @@
       </collision>
       <inertial>
-        <origin xyz="0.00 0.00 -0.12564" rpy="0 0 0" />
-        <mass value="0.2"/>
-        <inertia ixx="0.4201680" ixy="0" ixz="0" iyy="0.4196489" iyz="0" izz="0.0031965" />
+        <xacro:if value="${prefix == 'LF'}">
+          <origin xyz="-0.000162 -0.000597 -0.068453" rpy="0 0 0" />
+          <mass value="0.187"/>
+          <inertia ixx="0.001261336" ixy="0.000000011" ixz="-0.000001541" iyy="0.001259961" iyz="-0.0000059890" izz="0.000033267" />
+        </xacro:if>
+        <xacro:if value="${prefix == 'LH'}">
+          <origin xyz="-0.000162 -0.000597 -0.068453" rpy="0 0 0" />
+          <mass value="0.187"/>
+          <inertia ixx="0.001261336" ixy="0.000000011" ixz="-0.000001541" iyy="0.001259961" iyz="-0.0000059890" izz="0.000033267" />
+        </xacro:if>
+        <xacro:if value="${prefix == 'RH'}">
+          <origin xyz="-0.000162 0.000597 -0.068453" rpy="0 0 0" />
+          <mass value="0.187"/>
+          <inertia ixx="0.001261336" ixy="0.000000011" ixz="-0.000001541" iyy="0.001259961" iyz="-0.0000059890" izz="0.000033267" />
+        </xacro:if>
+        <xacro:if value="${prefix == 'RF'}">
+          <origin xyz="-0.000162 0.000597 -0.068453" rpy="0 0 0" />
+          <mass value="0.187"/>
+          <inertia ixx="0.001261336" ixy="0.000000011" ixz="-0.000001541" iyy="0.001259961" iyz="-0.0000059890" izz="0.000033267" />
+        </xacro:if>
       </inertial>
     </link>
