Commit message: update

File: orthrus_interfaces/models/orthrus/urdf/orthrus.urdf (robot description, URDF)
Before this commit: robot orthrus, 13 links, 12 joints
Links:
- removed link hip_LB
- removed link hip_LF
- removed link hip_RB
- removed link hip_RF
- removed link leg1_LB
- removed link leg1_LF
- removed link leg1_RB
- removed link leg1_RF
- removed link leg2_LB
- removed link leg2_LF
- removed link leg2_RB
- removed link leg2_RF
- added link HAA_LF, mass 0.7; collision mesh filename=file:////home/evence/code_file/ros2_ws/orthrus/install/orth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; visual mesh filename=file:////home/evence/code_file/ros2_ws/orthrus/install/orth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
- added link HAA_LH, mass 0.7; collision mesh filename=file:////home/evence/code_file/ros2_ws/orthrus/install/orth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; visual mesh filename=file:////home/evence/code_file/ros2_ws/orthrus/install/orth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
- added link HAA_RF, mass 0.7; collision mesh filename=file:////home/evence/code_file/ros2_ws/orthrus/install/orth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; visual mesh filename=file:////home/evence/code_file/ros2_ws/orthrus/install/orth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
- added link HAA_RH, mass 0.7; collision mesh filename=file:////home/evence/code_file/ros2_ws/orthrus/install/orth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; visual mesh filename=file:////home/evence/code_file/ros2_ws/orthrus/install/orth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
- added link HFE_LF, mass 1; collision mesh filename=file:////home/evence/code_file/ros2_ws/orthrus/install/orth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; visual mesh filename=file:////home/evence/code_file/ros2_ws/orthrus/install/orth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
- added link HFE_LH, mass 1; collision mesh filename=file:////home/evence/code_file/ros2_ws/orthrus/install/orth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; visual mesh filename=file:////home/evence/code_file/ros2_ws/orthrus/install/orth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
- added link HFE_RF, mass 1; collision mesh filename=file:////home/evence/code_file/ros2_ws/orthrus/install/orth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; visual mesh filename=file:////home/evence/code_file/ros2_ws/orthrus/install/orth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
- added link HFE_RH, mass 1; collision mesh filename=file:////home/evence/code_file/ros2_ws/orthrus/install/orth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; visual mesh filename=file:////home/evence/code_file/ros2_ws/orthrus/install/orth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
- added link KFE_LF, mass 0.2; collision mesh filename=file:////home/evence/code_file/ros2_ws/orthrus/install/orth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; visual mesh filename=file:////home/evence/code_file/ros2_ws/orthrus/install/orth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
- added link KFE_LH, mass 0.2; collision mesh filename=file:////home/evence/code_file/ros2_ws/orthrus/install/orth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; visual mesh filename=file:////home/evence/code_file/ros2_ws/orthrus/install/orth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
- added link KFE_RF, mass 0.2; collision mesh filename=file:////home/evence/code_file/ros2_ws/orthrus/install/orth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; visual mesh filename=file:////home/evence/code_file/ros2_ws/orthrus/install/orth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
- added link KFE_RH, mass 0.2; collision mesh filename=file:////home/evence/code_file/ros2_ws/orthrus/install/orth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; visual mesh filename=file:////home/evence/code_file/ros2_ws/orthrus/install/orth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
Joints:
- removed joint hip_LB_joint
- removed joint hip_LF_joint
- removed joint hip_RB_joint
- removed joint hip_RF_joint
- removed joint leg1_LB_joint
- removed joint leg1_LF_joint
- removed joint leg1_RB_joint
- removed joint leg1_RF_joint
- removed joint leg2_LB_joint
- removed joint leg2_LF_joint
- removed joint leg2_RB_joint
- removed joint leg2_RF_joint
- added joint HAA_LF_joint: type revolute, parent body, child HAA_LF, origin xyz=-0.05 0.20 0 rpy=1.5707963267948966 3.141592653589793 0, axis 0 0 1, limit lower=-1.5707963267948966 upper=1.5707963267948966 effort=35.0 velocity=3.141592653589793
- added joint HAA_LH_joint: type revolute, parent body, child HAA_LH, origin xyz=-0.05 -0.20 0 rpy=-1.5707963267948966 3.141592653589793 0, axis 0 0 1, limit lower=-1.5707963267948966 upper=1.5707963267948966 effort=35.0 velocity=3.141592653589793
- added joint HAA_RF_joint: type revolute, parent body, child HAA_RF, origin xyz=0.05 0.20 0 rpy=-1.5707963267948966 3.141592653589793 3.141592653589793, axis 0 0 1, limit lower=-1.5707963267948966 upper=1.5707963267948966 effort=35.0 velocity=3.141592653589793
- added joint HAA_RH_joint: type revolute, parent body, child HAA_RH, origin xyz=0.05 -0.20 0 rpy=1.5707963267948966 3.141592653589793 3.141592653589793, axis 0 0 1, limit lower=-1.5707963267948966 upper=1.5707963267948966 effort=35.0 velocity=3.141592653589793
- added joint HFE_LF_joint: type revolute, parent HAA_LF, child HFE_LF, origin xyz=0.05 0 0 rpy=-1.5707963267948966 0 0, axis 1 0 0, limit lower=-2.0943951023931953 upper=2.0943951023931953 effort=35.0 velocity=3.141592653589793
- added joint HFE_LH_joint: type revolute, parent HAA_LH, child HFE_LH, origin xyz=0.05 0 0 rpy=1.5707963267948966 0 0, axis 1 0 0, limit lower=-2.0943951023931953 upper=2.0943951023931953 effort=35.0 velocity=3.141592653589793
- added joint HFE_RF_joint: type revolute, parent HAA_RF, child HFE_RF, origin xyz=0.05 0 0 rpy=-1.5707963267948966 0 0, axis 1 0 0, limit lower=-2.0943951023931953 upper=2.0943951023931953 effort=35.0 velocity=3.141592653589793
- added joint HFE_RH_joint: type revolute, parent HAA_RH, child HFE_RH, origin xyz=0.05 0 0 rpy=1.5707963267948966 0 0, axis 1 0 0, limit lower=-2.0943951023931953 upper=2.0943951023931953 effort=35.0 velocity=3.141592653589793
- added joint KFE_LF_joint: type revolute, parent HFE_LF, child KFE_LF, origin xyz=0.035 -0.18 0 rpy=2.0943951023931953 0 0, axis 1 0 0, limit lower=-0.2617993877991494 upper=2.0943951023931953 effort=35.0 velocity=3.141592653589793
- added joint KFE_LH_joint: type revolute, parent HFE_LH, child KFE_LH, origin xyz=0.035 -0.18 0 rpy=2.0943951023931953 0 0, axis 1 0 0, limit lower=-0.2617993877991494 upper=2.0943951023931953 effort=35.0 velocity=3.141592653589793
- added joint KFE_RF_joint: type revolute, parent HFE_RF, child KFE_RF, origin xyz=0.035 -0.18 0 rpy=1.0471975511965976 0 0, axis 1 0 0, limit lower=-2.0943951023931953 upper=0.2617993877991494 effort=35.0 velocity=3.141592653589793
- added joint KFE_RH_joint: type revolute, parent HFE_RH, child KFE_RH, origin xyz=0.035 -0.18 0 rpy=1.0471975511965976 0 0, axis 1 0 0, limit lower=-2.0943951023931953 upper=0.2617993877991494 effort=35.0 velocity=3.141592653589793

File: orthrus_interfaces/models/orthrus/urdf/orthrus_base.xacro (robot description, xacro)
@@ -29,6 +29,6 @@
     </inertial>
   </link>
-  <xacro:macro name="hip" params="prefix">
-    <link name="hip_${prefix}">
+  <xacro:macro name="HAA" params="prefix">
+    <link name="HAA_${prefix}">
       <visual>
         <origin xyz="-0.02 -0.05 -0.05" rpy="0 0 0" />
@@ -49,8 +49,8 @@
       </inertial>
     </link>
-    <joint name="hip_${prefix}_joint" type="revolute">
+    <joint name="HAA_${prefix}_joint" type="revolute">
       <axis xyz="0 0 1"/>
       <parent link="body"/>
-      <child link="hip_${prefix}"/>
+      <child link="HAA_${prefix}"/>
       <dynamics damping="0.4" friction="0.3"/>
       <limit effort="35.0" lower="-${pi/2}" upper="${pi/2}" velocity="${pi}"/>
@@ -58,8 +58,8 @@
         <origin xyz="-0.05 0.20 0" rpy="${pi/2} ${pi} 0" />
       </xacro:if>
-      <xacro:if value="${prefix == 'LB'}">
+      <xacro:if value="${prefix == 'LH'}">
         <origin xyz="-0.05 -0.20 0" rpy="-${pi/2} ${pi} 0" />
       </xacro:if>
-      <xacro:if value="${prefix == 'RB'}">
+      <xacro:if value="${prefix == 'RH'}">
         <origin xyz="0.05 -0.20 0" rpy="${pi/2} ${pi} ${pi}" />
       </xacro:if>
@@ -69,6 +69,6 @@
     </joint>
   </xacro:macro>
-  <xacro:macro name="leg1" params="prefix">
-    <link name="leg1_${prefix}">
+  <xacro:macro name="HFE" params="prefix">
+    <link name="HFE_${prefix}">
       <visual>
         <origin xyz="0 -0.2 -0.05" rpy="0 0 0" />
@@ -89,8 +89,8 @@
       </inertial>
     </link>
-    <joint name="leg1_${prefix}_joint" type="revolute">
+    <joint name="HFE_${prefix}_joint" type="revolute">
       <axis xyz="1 0 0"/>
-      <parent link="hip_${prefix}"/>
-      <child link="leg1_${prefix}"/>
+      <parent link="HAA_${prefix}"/>
+      <child link="HFE_${prefix}"/>
       <dynamics damping="0.4" friction="0.3"/>
       <limit effort="35.0" lower="-${pi*2/3}" upper="${pi*2/3}" velocity="${pi}"/>
@@ -98,8 +98,8 @@
         <origin xyz="0.05 0 0" rpy="-${pi/2} 0 0" />
       </xacro:if>
-      <xacro:if value="${prefix == 'LB'}">
+      <xacro:if value="${prefix == 'LH'}">
         <origin xyz="0.05 0 0" rpy="${pi/2} 0 0" />
       </xacro:if>
-      <xacro:if value="${prefix == 'RB'}">
+      <xacro:if value="${prefix == 'RH'}">
         <origin xyz="0.05 0 0" rpy="${pi/2} 0 0" />
       </xacro:if>
@@ -109,6 +109,6 @@
     </joint>
   </xacro:macro>
-  <xacro:macro name="leg2" params="prefix">
-    <link name="leg2_${prefix}">
+  <xacro:macro name="KFE" params="prefix">
+    <link name="KFE_${prefix}">
       <visual>
         <origin xyz="-0.025 -0.025 -0.225" rpy="0 0 0" />
@@ -129,8 +129,8 @@
       </inertial>
     </link>
-    <joint name="leg2_${prefix}_joint" type="revolute">
+    <joint name="KFE_${prefix}_joint" type="revolute">
       <axis xyz="1 0 0"/>
-      <parent link="leg1_${prefix}"/>
-      <child link="leg2_${prefix}"/>
+      <parent link="HFE_${prefix}"/>
+      <child link="KFE_${prefix}"/>
       <dynamics damping="0.4" friction="0.3"/>
       <xacro:if value="${prefix == 'LF'}">
@@ -142,9 +142,9 @@
         <limit effort="35.0" lower="-${pi*2/3}" upper="${pi*1/12}" velocity="${pi}"/>
       </xacro:if>
-      <xacro:if value="${prefix == 'RB'}">
+      <xacro:if value="${prefix == 'RH'}">
         <origin xyz="0.035 -0.18 0" rpy="${pi*1/3} 0 0" />
         <limit effort="35.0" lower="-${pi*2/3}" upper="${pi*1/12}" velocity="${pi}"/>
       </xacro:if>
-      <xacro:if value="${prefix == 'LB'}">
+      <xacro:if value="${prefix == 'LH'}">
         <origin xyz="0.035 -0.18 0" rpy="${pi*2/3} 0 0" />
         <limit effort="35.0" lower="-${pi*1/12}" upper="${pi*2/3}" velocity="${pi}"/>
@@ -152,6 +152,6 @@
     </joint>
   </xacro:macro>
-  <xacro:macro name="ros2_hip_joint" params="prefix">
-    <joint name="hip_${prefix}_joint">
+  <xacro:macro name="ros2_HAA_joint" params="prefix">
+    <joint name="HAA_${prefix}_joint">
       <command_interface name="effort">
         <param name="min">-35</param>
@@ -163,6 +163,6 @@
     </joint>
   </xacro:macro>
-  <xacro:macro name="ros2_leg1_joint" params="prefix">
-    <joint name="leg1_${prefix}_joint">
+  <xacro:macro name="ros2_HFE_joint" params="prefix">
+    <joint name="HFE_${prefix}_joint">
       <command_interface name="effort">
         <param name="min">-35</param>
@@ -174,6 +174,6 @@
     </joint>
   </xacro:macro>
-  <xacro:macro name="ros2_leg2_joint" params="prefix">
-    <joint name="leg2_${prefix}_joint">
+  <xacro:macro name="ros2_KFE_joint" params="prefix">
+    <joint name="KFE_${prefix}_joint">
       <command_interface name="effort">
         <param name="min">-35</param>

File: orthrus_interfaces/models/orthrus/urdf/orthrus_for_gazebo.urdf.xacro (robot description, xacro)
@@ -3,16 +3,16 @@
   xmlns:xacro="http://ros.org/wiki/xacro">
   <xacro:include filename="orthrus_base.xacro"/>
-  <xacro:hip prefix="RF"/>
-  <xacro:hip prefix="LF"/>
-  <xacro:hip prefix="RB"/>
-  <xacro:hip prefix="LB"/>
-  <xacro:leg1 prefix="RF"/>
-  <xacro:leg1 prefix="LF"/>
-  <xacro:leg1 prefix="RB"/>
-  <xacro:leg1 prefix="LB"/>
-  <xacro:leg2 prefix="LF"/>
-  <xacro:leg2 prefix="RF"/>
-  <xacro:leg2 prefix="LB"/>
-  <xacro:leg2 prefix="RB"/>
+  <xacro:HAA prefix="RF"/>
+  <xacro:HAA prefix="LF"/>
+  <xacro:HAA prefix="RH"/>
+  <xacro:HAA prefix="LH"/>
+  <xacro:HFE prefix="RF"/>
+  <xacro:HFE prefix="LF"/>
+  <xacro:HFE prefix="RH"/>
+  <xacro:HFE prefix="LH"/>
+  <xacro:KFE prefix="LF"/>
+  <xacro:KFE prefix="RF"/>
+  <xacro:KFE prefix="LH"/>
+  <xacro:KFE prefix="RH"/>
   <gazebo reference="body">
     <sensor name="imu_sensor" type="imu">
@@ -25,16 +25,16 @@
       <plugin>gazebo_ros2_control/GazeboSystem</plugin>
     </hardware>
-    <xacro:ros2_hip_joint prefix="RF"/>
-    <xacro:ros2_leg1_joint prefix="RF"/>
-    <xacro:ros2_leg2_joint prefix="RF"/>
-    <xacro:ros2_hip_joint prefix="LF"/>
-    <xacro:ros2_leg1_joint prefix="LF"/>
-    <xacro:ros2_leg2_joint prefix="LF"/>
-    <xacro:ros2_hip_joint prefix="RB"/>
-    <xacro:ros2_leg1_joint prefix="RB"/>
-    <xacro:ros2_leg2_joint prefix="RB"/>
-    <xacro:ros2_hip_joint prefix="LB"/>
-    <xacro:ros2_leg1_joint prefix="LB"/>
-    <xacro:ros2_leg2_joint prefix="LB"/>
+    <xacro:ros2_HAA_joint prefix="RF"/>
+    <xacro:ros2_HFE_joint prefix="RF"/>
+    <xacro:ros2_KFE_joint prefix="RF"/>
+    <xacro:ros2_HAA_joint prefix="LF"/>
+    <xacro:ros2_HFE_joint prefix="LF"/>
+    <xacro:ros2_KFE_joint prefix="LF"/>
+    <xacro:ros2_HAA_joint prefix="RH"/>
+    <xacro:ros2_HFE_joint prefix="RH"/>
+    <xacro:ros2_KFE_joint prefix="RH"/>
+    <xacro:ros2_HAA_joint prefix="LH"/>
+    <xacro:ros2_HFE_joint prefix="LH"/>
+    <xacro:ros2_KFE_joint prefix="LH"/>
     <sensor name="imu_sensor">
       <state_interface name="orientation.x"/>

Commit message: update

File: orthrus_interfaces/models/orthrus/urdf/orthrus.urdf (robot description, URDF)
Before this commit: robot orthrus, 13 links, 12 joints
Links:
- removed link HAA_LF
- removed link HAA_LH
- removed link HAA_RF
- removed link HAA_RH
- removed link HFE_LF
- removed link HFE_LH
- removed link HFE_RF
- removed link HFE_RH
- removed link KFE_LF
- removed link KFE_LH
- removed link KFE_RF
- removed link KFE_RH
- added link LF_HAA, mass 0.7; collision mesh filename=file:////home/evence/code_file/ros2_ws/orthrus/install/orth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; visual mesh filename=file:////home/evence/code_file/ros2_ws/orthrus/install/orth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
- added link LF_HFE, mass 1; collision mesh filename=file:////home/evence/code_file/ros2_ws/orthrus/install/orth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; visual mesh filename=file:////home/evence/code_file/ros2_ws/orthrus/install/orth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
- added link LF_KFE, mass 0.2; collision mesh filename=file:////home/evence/code_file/ros2_ws/orthrus/install/orth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; visual mesh filename=file:////home/evence/code_file/ros2_ws/orthrus/install/orth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
- added link LH_HAA, mass 0.7; collision mesh filename=file:////home/evence/code_file/ros2_ws/orthrus/install/orth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; visual mesh filename=file:////home/evence/code_file/ros2_ws/orthrus/install/orth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
- added link LH_HFE, mass 1; collision mesh filename=file:////home/evence/code_file/ros2_ws/orthrus/install/orth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; visual mesh filename=file:////home/evence/code_file/ros2_ws/orthrus/install/orth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
- added link LH_KFE, mass 0.2; collision mesh filename=file:////home/evence/code_file/ros2_ws/orthrus/install/orth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; visual mesh filename=file:////home/evence/code_file/ros2_ws/orthrus/install/orth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
- added link RF_HAA, mass 0.7; collision mesh filename=file:////home/evence/code_file/ros2_ws/orthrus/install/orth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; visual mesh filename=file:////home/evence/code_file/ros2_ws/orthrus/install/orth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
- added link RF_HFE, mass 1; collision mesh filename=file:////home/evence/code_file/ros2_ws/orthrus/install/orth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; visual mesh filename=file:////home/evence/code_file/ros2_ws/orthrus/install/orth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
- added link RF_KFE, mass 0.2; collision mesh filename=file:////home/evence/code_file/ros2_ws/orthrus/install/orth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; visual mesh filename=file:////home/evence/code_file/ros2_ws/orthrus/install/orth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
- added link RH_HAA, mass 0.7; collision mesh filename=file:////home/evence/code_file/ros2_ws/orthrus/install/orth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; visual mesh filename=file:////home/evence/code_file/ros2_ws/orthrus/install/orth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
- added link RH_HFE, mass 1; collision mesh filename=file:////home/evence/code_file/ros2_ws/orthrus/install/orth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; visual mesh filename=file:////home/evence/code_file/ros2_ws/orthrus/install/orth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
- added link RH_KFE, mass 0.2; collision mesh filename=file:////home/evence/code_file/ros2_ws/orthrus/install/orth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; visual mesh filename=file:////home/evence/code_file/ros2_ws/orthrus/install/orth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
Joints:
- removed joint HAA_LF_joint
- removed joint HAA_LH_joint
- removed joint HAA_RF_joint
- removed joint HAA_RH_joint
- removed joint HFE_LF_joint
- removed joint HFE_LH_joint
- removed joint HFE_RF_joint
- removed joint HFE_RH_joint
- removed joint KFE_LF_joint
- removed joint KFE_LH_joint
- removed joint KFE_RF_joint
- removed joint KFE_RH_joint
- added joint LF_HAA: type revolute, parent body, child LF_HAA, origin xyz=-0.05 0.20 0 rpy=1.5707963267948966 3.141592653589793 0, axis 0 0 1, limit lower=-1.5707963267948966 upper=1.5707963267948966 effort=35.0 velocity=3.141592653589793
- added joint LF_HFE: type revolute, parent LF_HAA, child LF_HFE, origin xyz=0.05 0 0 rpy=-1.5707963267948966 0 0, axis 1 0 0, limit lower=-2.0943951023931953 upper=2.0943951023931953 effort=35.0 velocity=3.141592653589793
- added joint LF_KFE: type revolute, parent LF_HFE, child LF_KFE, origin xyz=0.035 -0.18 0 rpy=2.0943951023931953 0 0, axis 1 0 0, limit lower=-0.2617993877991494 upper=2.0943951023931953 effort=35.0 velocity=3.141592653589793
- added joint LH_HAA: type revolute, parent body, child LH_HAA, origin xyz=-0.05 -0.20 0 rpy=-1.5707963267948966 3.141592653589793 0, axis 0 0 1, limit lower=-1.5707963267948966 upper=1.5707963267948966 effort=35.0 velocity=3.141592653589793
- added joint LH_HFE: type revolute, parent LH_HAA, child LH_HFE, origin xyz=0.05 0 0 rpy=1.5707963267948966 0 0, axis 1 0 0, limit lower=-2.0943951023931953 upper=2.0943951023931953 effort=35.0 velocity=3.141592653589793
- added joint LH_KFE: type revolute, parent LH_HFE, child LH_KFE, origin xyz=0.035 -0.18 0 rpy=2.0943951023931953 0 0, axis 1 0 0, limit lower=-0.2617993877991494 upper=2.0943951023931953 effort=35.0 velocity=3.141592653589793
- added joint RF_HAA: type revolute, parent body, child RF_HAA, origin xyz=0.05 0.20 0 rpy=-1.5707963267948966 3.141592653589793 3.141592653589793, axis 0 0 1, limit lower=-1.5707963267948966 upper=1.5707963267948966 effort=35.0 velocity=3.141592653589793
- added joint RF_HFE: type revolute, parent RF_HAA, child RF_HFE, origin xyz=0.05 0 0 rpy=-1.5707963267948966 0 0, axis 1 0 0, limit lower=-2.0943951023931953 upper=2.0943951023931953 effort=35.0 velocity=3.141592653589793
- added joint RF_KFE: type revolute, parent RF_HFE, child RF_KFE, origin xyz=0.035 -0.18 0 rpy=1.0471975511965976 0 0, axis 1 0 0, limit lower=-2.0943951023931953 upper=0.2617993877991494 effort=35.0 velocity=3.141592653589793
- added joint RH_HAA: type revolute, parent body, child RH_HAA, origin xyz=0.05 -0.20 0 rpy=1.5707963267948966 3.141592653589793 3.141592653589793, axis 0 0 1, limit lower=-1.5707963267948966 upper=1.5707963267948966 effort=35.0 velocity=3.141592653589793
- added joint RH_HFE: type revolute, parent RH_HAA, child RH_HFE, origin xyz=0.05 0 0 rpy=1.5707963267948966 0 0, axis 1 0 0, limit lower=-2.0943951023931953 upper=2.0943951023931953 effort=35.0 velocity=3.141592653589793
- added joint RH_KFE: type revolute, parent RH_HFE, child RH_KFE, origin xyz=0.035 -0.18 0 rpy=1.0471975511965976 0 0, axis 1 0 0, limit lower=-2.0943951023931953 upper=0.2617993877991494 effort=35.0 velocity=3.141592653589793

File: orthrus_interfaces/models/orthrus/urdf/orthrus_base.xacro (robot description, xacro)
@@ -30,5 +30,5 @@
   </link>
   <xacro:macro name="HAA" params="prefix">
-    <link name="HAA_${prefix}">
+    <link name="${prefix}_HAA">
       <visual>
         <origin xyz="-0.02 -0.05 -0.05" rpy="0 0 0" />
@@ -49,8 +49,8 @@
       </inertial>
     </link>
-    <joint name="HAA_${prefix}_joint" type="revolute">
+    <joint name="${prefix}_HAA" type="revolute">
       <axis xyz="0 0 1"/>
       <parent link="body"/>
-      <child link="HAA_${prefix}"/>
+      <child link="${prefix}_HAA"/>
       <dynamics damping="0.4" friction="0.3"/>
       <limit effort="35.0" lower="-${pi/2}" upper="${pi/2}" velocity="${pi}"/>
@@ -70,5 +70,5 @@
   </xacro:macro>
   <xacro:macro name="HFE" params="prefix">
-    <link name="HFE_${prefix}">
+    <link name="${prefix}_HFE">
       <visual>
         <origin xyz="0 -0.2 -0.05" rpy="0 0 0" />
@@ -89,8 +89,8 @@
       </inertial>
     </link>
-    <joint name="HFE_${prefix}_joint" type="revolute">
+    <joint name="${prefix}_HFE" type="revolute">
       <axis xyz="1 0 0"/>
-      <parent link="HAA_${prefix}"/>
-      <child link="HFE_${prefix}"/>
+      <parent link="${prefix}_HAA"/>
+      <child link="${prefix}_HFE"/>
       <dynamics damping="0.4" friction="0.3"/>
       <limit effort="35.0" lower="-${pi*2/3}" upper="${pi*2/3}" velocity="${pi}"/>
@@ -110,5 +110,5 @@
   </xacro:macro>
   <xacro:macro name="KFE" params="prefix">
-    <link name="KFE_${prefix}">
+    <link name="${prefix}_KFE">
       <visual>
         <origin xyz="-0.025 -0.025 -0.225" rpy="0 0 0" />
@@ -129,8 +129,8 @@
       </inertial>
     </link>
-    <joint name="KFE_${prefix}_joint" type="revolute">
+    <joint name="${prefix}_KFE" type="revolute">
       <axis xyz="1 0 0"/>
-      <parent link="HFE_${prefix}"/>
-      <child link="KFE_${prefix}"/>
+      <parent link="${prefix}_HFE"/>
+      <child link="${prefix}_KFE"/>
       <dynamics damping="0.4" friction="0.3"/>
       <xacro:if value="${prefix == 'LF'}">
