Commit message: update

File: orthrus_interfaces/models/orthrus/urdf/orthrus.urdf (robot description, URDF)
Before this commit: robot orthrus, 13 links, 12 joints
Links:
- removed link body
- added link base, mass 7; collision mesh filename=file:///home/evence/code_file/ros2_ws/orthrus/install/orthr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; visual mesh filename=file:///home/evence/code_file/ros2_ws/orthrus/install/orthr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
- link LF_HAA: geometry collision mesh filename=file:///home/evence/code_file/ros2_ws/orthrus/install/orthr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; visual mesh filename=file:///home/evence/code_file/ros2_ws/orthrus/install/orthr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
- link LF_HFE: geometry collision mesh filename=file:///home/evence/code_file/ros2_ws/orthrus/install/orthr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; visual mesh filename=file:///home/evence/code_file/ros2_ws/orthrus/install/orthr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
- link LF_KFE: geometry collision mesh filename=file:///home/evence/code_file/ros2_ws/orthrus/install/orthr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; visual mesh filename=file:///home/evence/code_file/ros2_ws/orthrus/install/orthr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
- link LH_HAA: geometry collision mesh filename=file:///home/evence/code_file/ros2_ws/orthrus/install/orthr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; visual mesh filename=file:///home/evence/code_file/ros2_ws/orthrus/install/orthr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
- link LH_HFE: geometry collision mesh filename=file:///home/evence/code_file/ros2_ws/orthrus/install/orthr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; visual mesh filename=file:///home/evence/code_file/ros2_ws/orthrus/install/orthr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
- link LH_KFE: geometry collision mesh filename=file:///home/evence/code_file/ros2_ws/orthrus/install/orthr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; visual mesh filename=file:///home/evence/code_file/ros2_ws/orthrus/install/orthr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
- link RF_HAA: geometry collision mesh filename=file:///home/evence/code_file/ros2_ws/orthrus/install/orthr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; visual mesh filename=file:///home/evence/code_file/ros2_ws/orthrus/install/orthr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
- link RF_HFE: geometry collision mesh filename=file:///home/evence/code_file/ros2_ws/orthrus/install/orthr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; visual mesh filename=file:///home/evence/code_file/ros2_ws/orthrus/install/orthr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
- link RF_KFE: geometry collision mesh filename=file:///home/evence/code_file/ros2_ws/orthrus/install/orthr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; visual mesh filename=file:///home/evence/code_file/ros2_ws/orthrus/install/orthr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
- link RH_HAA: geometry collision mesh filename=file:///home/evence/code_file/ros2_ws/orthrus/install/orthr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; visual mesh filename=file:///home/evence/code_file/ros2_ws/orthrus/install/orthr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
- link RH_HFE: geometry collision mesh filename=file:///home/evence/code_file/ros2_ws/orthrus/install/orthr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; visual mesh filename=file:///home/evence/code_file/ros2_ws/orthrus/install/orthr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
- link RH_KFE: geometry collision mesh filename=file:///home/evence/code_file/ros2_ws/orthrus/install/orthr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; visual mesh filename=file:///home/evence/code_file/ros2_ws/orthrus/install/orthr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
Joints:
- joint LF_HAA: parent body -> base
- joint LH_HAA: parent body -> base
- joint RF_HAA: parent body -> base
- joint RH_HAA: parent body -> base

File: orthrus_interfaces/models/orthrus/urdf/orthrus_base.xacro (robot description, xacro)
@@ -1,4 +1,4 @@
 <robot name="orthrus_base" xmlns:xacro="http://ros.org/wiki/xacro">
-  <xacro:property name="meshes_folder" value="file:///$(find orthrus_gazebo)/models/orthrus/meshes" />
+  <xacro:property name="meshes_folder" value="file://$(find orthrus_gazebo)/models/orthrus/meshes" />
   <material name="blue">
     <color rgba="0 0 0.8 1"/>
@@ -10,5 +10,5 @@
     <color rgba="1 1 1 1"/>
   </material>
-  <link name="body">
+  <link name="base">
     <visual>
       <origin xyz="-0.10 0.1385 -0.05" rpy="${pi/2} 0 0" />
@@ -51,5 +51,5 @@
     <joint name="${prefix}_HAA" type="revolute">
       <axis xyz="0 0 1"/>
-      <parent link="body"/>
+      <parent link="base"/>
       <child link="${prefix}_HAA"/>
       <dynamics damping="0.4" friction="0.3"/>

Commit message: update

File: orthrus_interfaces/models/orthrus/urdf/orthrus.urdf (robot description, URDF)
Before this commit: robot orthrus, 13 links, 12 joints
Links:
- link LF_HAA: geometry collision mesh filename=file:////home/evence/code_file/ros2_ws/orthrus/install/orth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; visual mesh filename=file:////home/evence/code_file/ros2_ws/orthrus/install/orth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
- link LF_HFE: geometry collision mesh filename=file:////home/evence/code_file/ros2_ws/orthrus/install/orth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; visual mesh filename=file:////home/evence/code_file/ros2_ws/orthrus/install/orth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
- link LF_KFE: geometry collision mesh filename=file:////home/evence/code_file/ros2_ws/orthrus/install/orth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; visual mesh filename=file:////home/evence/code_file/ros2_ws/orthrus/install/orth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
- link LH_HAA: geometry collision mesh filename=file:////home/evence/code_file/ros2_ws/orthrus/install/orth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; visual mesh filename=file:////home/evence/code_file/ros2_ws/orthrus/install/orth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
- link LH_HFE: geometry collision mesh filename=file:////home/evence/code_file/ros2_ws/orthrus/install/orth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; visual mesh filename=file:////home/evence/code_file/ros2_ws/orthrus/install/orth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
- link LH_KFE: geometry collision mesh filename=file:////home/evence/code_file/ros2_ws/orthrus/install/orth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; visual mesh filename=file:////home/evence/code_file/ros2_ws/orthrus/install/orth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
- link RF_HAA: geometry collision mesh filename=file:////home/evence/code_file/ros2_ws/orthrus/install/orth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; visual mesh filename=file:////home/evence/code_file/ros2_ws/orthrus/install/orth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
- link RF_HFE: geometry collision mesh filename=file:////home/evence/code_file/ros2_ws/orthrus/install/orth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; visual mesh filename=file:////home/evence/code_file/ros2_ws/orthrus/install/orth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
- link RF_KFE: geometry collision mesh filename=file:////home/evence/code_file/ros2_ws/orthrus/install/orth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; visual mesh filename=file:////home/evence/code_file/ros2_ws/orthrus/install/orth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
- link RH_HAA: geometry collision mesh filename=file:////home/evence/code_file/ros2_ws/orthrus/install/orth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; visual mesh filename=file:////home/evence/code_file/ros2_ws/orthrus/install/orth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
- link RH_HFE: geometry collision mesh filename=file:////home/evence/code_file/ros2_ws/orthrus/install/orth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; visual mesh filename=file:////home/evence/code_file/ros2_ws/orthrus/install/orth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
- link RH_KFE: geometry collision mesh filename=file:////home/evence/code_file/ros2_ws/orthrus/install/orth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; visual mesh filename=file:////home/evence/code_file/ros2_ws/orthrus/install/orth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
- link base: geometry collision mesh filename=file:////home/evence/code_file/ros2_ws/orthrus/install/orth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; visual mesh filename=file:////home/evence/code_file/ros2_ws/orthrus/install/orth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

File: orthrus_interfaces/models/orthrus/urdf/orthrus.urdf.xacro (robot description, xacro)
@@ -2,4 +2,5 @@
 <robot name="orthrus"
   xmlns:xacro="http://ros.org/wiki/xacro">
+  <xacro:property name="meshes_folder" value="file:///$(find orthrus_gazebo)/models/orthrus/meshes" />
   <xacro:include filename="orthrus_base.xacro"/>
   <xacro:HAA prefix="RF"/>

File: orthrus_interfaces/models/orthrus/urdf/orthrus_base.xacro (robot description, xacro)
@@ -1,4 +1,3 @@
 <robot name="orthrus_base" xmlns:xacro="http://ros.org/wiki/xacro">
-  <xacro:property name="meshes_folder" value="file://$(find orthrus_gazebo)/models/orthrus/meshes" />
   <material name="blue">
     <color rgba="0 0 0.8 1"/>

File: orthrus_interfaces/models/orthrus/urdf/orthrus_for_gazebo.urdf.xacro (robot description, xacro)
@@ -2,4 +2,5 @@
 <robot name="orthrus"
   xmlns:xacro="http://ros.org/wiki/xacro">
+  <xacro:property name="meshes_folder" value="file:///$(find orthrus_gazebo)/models/orthrus/meshes" />
   <xacro:include filename="orthrus_base.xacro"/>
   <xacro:HAA prefix="RF"/>

Commit message: update

File: orthrus_interfaces/models/orthrus/urdf/orthrus.urdf (robot description, URDF)
Before this commit: robot orthrus, 13 links, 12 joints
Links:
- removed link LF_HAA
- removed link LF_HFE
- removed link LF_KFE
- removed link LH_HAA
- removed link LH_HFE
- removed link LH_KFE
- removed link RF_HAA
- removed link RF_HFE
- removed link RF_KFE
- removed link RH_HAA
- removed link RH_HFE
- removed link RH_KFE
- added link LF_HAA_link, mass 0.7; collision mesh filename=file:////home/evence/code_file/ros2_ws/orthrus/install/orth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; visual mesh filename=file:////home/evence/code_file/ros2_ws/orthrus/install/orth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
- added link LF_HFE_link, mass 1; collision mesh filename=file:////home/evence/code_file/ros2_ws/orthrus/install/orth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; visual mesh filename=file:////home/evence/code_file/ros2_ws/orthrus/install/orth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
- added link LF_KFE_link, mass 0.2; collision mesh filename=file:////home/evence/code_file/ros2_ws/orthrus/install/orth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; visual mesh filename=file:////home/evence/code_file/ros2_ws/orthrus/install/orth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
- added link LH_HAA_link, mass 0.7; collision mesh filename=file:////home/evence/code_file/ros2_ws/orthrus/install/orth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; visual mesh filename=file:////home/evence/code_file/ros2_ws/orthrus/install/orth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
- added link LH_HFE_link, mass 1; collision mesh filename=file:////home/evence/code_file/ros2_ws/orthrus/install/orth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; visual mesh filename=file:////home/evence/code_file/ros2_ws/orthrus/install/orth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
- added link LH_KFE_link, mass 0.2; collision mesh filename=file:////home/evence/code_file/ros2_ws/orthrus/install/orth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; visual mesh filename=file:////home/evence/code_file/ros2_ws/orthrus/install/orth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
- added link RF_HAA_link, mass 0.7; collision mesh filename=file:////home/evence/code_file/ros2_ws/orthrus/install/orth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; visual mesh filename=file:////home/evence/code_file/ros2_ws/orthrus/install/orth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
- added link RF_HFE_link, mass 1; collision mesh filename=file:////home/evence/code_file/ros2_ws/orthrus/install/orth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; visual mesh filename=file:////home/evence/code_file/ros2_ws/orthrus/install/orth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
- added link RF_KFE_link, mass 0.2; collision mesh filename=file:////home/evence/code_file/ros2_ws/orthrus/install/orth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; visual mesh filename=file:////home/evence/code_file/ros2_ws/orthrus/install/orth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
- added link RH_HAA_link, mass 0.7; collision mesh filename=file:////home/evence/code_file/ros2_ws/orthrus/install/orth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; visual mesh filename=file:////home/evence/code_file/ros2_ws/orthrus/install/orth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
- added link RH_HFE_link, mass 1; collision mesh filename=file:////home/evence/code_file/ros2_ws/orthrus/install/orth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; visual mesh filename=file:////home/evence/code_file/ros2_ws/orthrus/install/orth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
- added link RH_KFE_link, mass 0.2; collision mesh filename=file:////home/evence/code_file/ros2_ws/orthrus/install/orth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; visual mesh filename=file:////home/evence/code_file/ros2_ws/orthrus/install/orth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
Joints:
- joint LF_HAA: child LF_HAA -> LF_HAA_link
- joint LF_HFE: child LF_HFE -> LF_HFE_link; parent LF_HAA -> LF_HAA_link
- joint LF_KFE: child LF_KFE -> LF_KFE_link; parent LF_HFE -> LF_HFE_link
- joint LH_HAA: child LH_HAA -> LH_HAA_link
- joint LH_HFE: child LH_HFE -> LH_HFE_link; parent LH_HAA -> LH_HAA_link
- joint LH_KFE: child LH_KFE -> LH_KFE_link; parent LH_HFE -> LH_HFE_link
- joint RF_HAA: child RF_HAA -> RF_HAA_link
- joint RF_HFE: child RF_HFE -> RF_HFE_link; parent RF_HAA -> RF_HAA_link
- joint RF_KFE: child RF_KFE -> RF_KFE_link; parent RF_HFE -> RF_HFE_link
- joint RH_HAA: child RH_HAA -> RH_HAA_link
- joint RH_HFE: child RH_HFE -> RH_HFE_link; parent RH_HAA -> RH_HAA_link
- joint RH_KFE: child RH_KFE -> RH_KFE_link; parent RH_HFE -> RH_HFE_link

Commit message: update

File: orthrus_interfaces/models/orthrus/urdf/orthrus.urdf (robot description, URDF)
Before this commit: robot orthrus, 13 links, 12 joints
Links:
- link LF_HAA_link: geometry collision mesh filename=file:////home/orthrus/orthrus/install/orthrus_interfaces/sh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; visual mesh filename=file:////home/orthrus/orthrus/install/orthrus_interfaces/sh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
- link LF_HFE_link: geometry collision mesh filename=file:////home/orthrus/orthrus/install/orthrus_interfaces/sh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; visual mesh filename=file:////home/orthrus/orthrus/install/orthrus_interfaces/sh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
- link LF_KFE_link: geometry collision mesh filename=file:////home/orthrus/orthrus/install/orthrus_interfaces/sh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; visual mesh filename=file:////home/orthrus/orthrus/install/orthrus_interfaces/sh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
- link LH_HAA_link: geometry collision mesh filename=file:////home/orthrus/orthrus/install/orthrus_interfaces/sh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; visual mesh filename=file:////home/orthrus/orthrus/install/orthrus_interfaces/sh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
- link LH_HFE_link: geometry collision mesh filename=file:////home/orthrus/orthrus/install/orthrus_interfaces/sh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; visual mesh filename=file:////home/orthrus/orthrus/install/orthrus_interfaces/sh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
- link LH_KFE_link: geometry collision mesh filename=file:////home/orthrus/orthrus/install/orthrus_interfaces/sh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; visual mesh filename=file:////home/orthrus/orthrus/install/orthrus_interfaces/sh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
- link RF_HAA_link: geometry collision mesh filename=file:////home/orthrus/orthrus/install/orthrus_interfaces/sh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; visual mesh filename=file:////home/orthrus/orthrus/install/orthrus_interfaces/sh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
- link RF_HFE_link: geometry collision mesh filename=file:////home/orthrus/orthrus/install/orthrus_interfaces/sh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; visual mesh filename=file:////home/orthrus/orthrus/install/orthrus_interfaces/sh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
- link RF_KFE_link: geometry collision mesh filename=file:////home/orthrus/orthrus/install/orthrus_interfaces/sh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; visual mesh filename=file:////home/orthrus/orthrus/install/orthrus_interfaces/sh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
- link RH_HAA_link: geometry collision mesh filename=file:////home/orthrus/orthrus/install/orthrus_interfaces/sh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; visual mesh filename=file:////home/orthrus/orthrus/install/orthrus_interfaces/sh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
- link RH_HFE_link: geometry collision mesh filename=file:////home/orthrus/orthrus/install/orthrus_interfaces/sh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; visual mesh filename=file:////home/orthrus/orthrus/install/orthrus_interfaces/sh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
- link RH_KFE_link: geometry collision mesh filename=file:////home/orthrus/orthrus/install/orthrus_interfaces/sh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; visual mesh filename=file:////home/orthrus/orthrus/install/orthrus_interfaces/sh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
- link base: geometry collision mesh filename=file:////home/orthrus/orthrus/install/orthrus_interfaces/sh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; visual mesh filename=file:////home/orthrus/orthrus/install/orthrus_interfaces/sh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

File: orthrus_interfaces/models/orthrus/urdf/orthrus.urdf.xacro (robot description, xacro)
@@ -53,5 +53,5 @@
   <gazebo>
     <plugin filename="libgazebo_ros2_control.so" name="gazebo_ros2_control">
-      <parameters>/home/evence/code_file/ros2_ws/orthrus/src/orthrus_ros2_pack/orthrus_sim/orthrus_gazebo/config/orthrus.yaml</parameters>
+      <parameters>/home/orthrus/orthrus/src/orthrus_ros2_pack/orthrus_sim/orthrus_gazebo/config/orthrus.yaml</parameters>
     </plugin>
   </gazebo>

Commit message: update

File: orthrus_interfaces/models/orthrus/urdf/orthrus.urdf (robot description, URDF)
Before this commit: robot orthrus, 13 links, 12 joints
Links:
- link LF_HAA_link: geometry collision mesh filename=file:////home/evence/code_file/ros2_ws/orthrus/install/orth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; visual mesh filename=file:////home/evence/code_file/ros2_ws/orthrus/install/orth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
- link LF_HFE_link: geometry collision mesh filename=file:////home/evence/code_file/ros2_ws/orthrus/install/orth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; visual mesh filename=file:////home/evence/code_file/ros2_ws/orthrus/install/orth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
- link LF_KFE_link: geometry collision mesh filename=file:////home/evence/code_file/ros2_ws/orthrus/install/orth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; visual mesh filename=file:////home/evence/code_file/ros2_ws/orthrus/install/orth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
- link LH_HAA_link: geometry collision mesh filename=file:////home/evence/code_file/ros2_ws/orthrus/install/orth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; visual mesh filename=file:////home/evence/code_file/ros2_ws/orthrus/install/orth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
- link LH_HFE_link: geometry collision mesh filename=file:////home/evence/code_file/ros2_ws/orthrus/install/orth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; visual mesh filename=file:////home/evence/code_file/ros2_ws/orthrus/install/orth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
- link LH_KFE_link: geometry collision mesh filename=file:////home/evence/code_file/ros2_ws/orthrus/install/orth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; visual mesh filename=file:////home/evence/code_file/ros2_ws/orthrus/install/orth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
- link RF_HAA_link: geometry collision mesh filename=file:////home/evence/code_file/ros2_ws/orthrus/install/orth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; visual mesh filename=file:////home/evence/code_file/ros2_ws/orthrus/install/orth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
- link RF_HFE_link: geometry collision mesh filename=file:////home/evence/code_file/ros2_ws/orthrus/install/orth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; visual mesh filename=file:////home/evence/code_file/ros2_ws/orthrus/install/orth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
- link RF_KFE_link: geometry collision mesh filename=file:////home/evence/code_file/ros2_ws/orthrus/install/orth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; visual mesh filename=file:////home/evence/code_file/ros2_ws/orthrus/install/orth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
- link RH_HAA_link: geometry collision mesh filename=file:////home/evence/code_file/ros2_ws/orthrus/install/orth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; visual mesh filename=file:////home/evence/code_file/ros2_ws/orthrus/install/orth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
- link RH_HFE_link: geometry collision mesh filename=file:////home/evence/code_file/ros2_ws/orthrus/install/orth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; visual mesh filename=file:////home/evence/code_file/ros2_ws/orthrus/install/orth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
- link RH_KFE_link: geometry collision mesh filename=file:////home/evence/code_file/ros2_ws/orthrus/install/orth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; visual mesh filename=file:////home/evence/code_file/ros2_ws/orthrus/install/orth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
- link base: geometry collision mesh filename=file:////home/evence/code_file/ros2_ws/orthrus/install/orth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; visual mesh filename=file:////home/evence/code_file/ros2_ws/orthrus/install/orth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

File: orthrus_interfaces/models/orthrus/urdf/orthrus.urdf.xacro (robot description, xacro)
@@ -53,5 +53,5 @@
   <gazebo>
     <plugin filename="libgazebo_ros2_control.so" name="gazebo_ros2_control">
-      <parameters>/home/orthrus/orthrus/src/orthrus_ros2_pack/orthrus_sim/orthrus_gazebo/config/orthrus.yaml</parameters>
+      <parameters>/home/evence/code_file/ros2_ws/orthrus/src/orthrus_ros2_pack/orthrus_sim/orthrus_gazebo/config/orthrus.yaml</parameters>
     </plugin>
   </gazebo>

Commit message: update

File: orthrus_interfaces/models/orthrus/urdf/orthrus.urdf (robot description, URDF)
Before this commit: robot orthrus, 13 links, 12 joints
Joints:
- joint LF_HAA: origin xyz=-0.05 0.20 0 rpy=1.5707963267948966 3.141592653589793 0 -> xyz=0.20 0.05 0 rpy=1.5707963267948966 3.141592653589793 -1.5707963267948966
- joint LH_HAA: origin xyz=-0.05 -0.20 0 rpy=-1.5707963267948966 3.141592653589793 0 -> xyz=-0.20 0.05 0 rpy=-1.5707963267948966 3.141592653589793 -1.5707963267948966
- joint RF_HAA: origin xyz=0.05 0.20 0 rpy=-1.5707963267948966 3.141592653589793 3.141592653589793 -> xyz=0.20 -0.05 0 rpy=-1.5707963267948966 3.141592653589793 1.5707963267948966
- joint RH_HAA: origin xyz=0.05 -0.20 0 rpy=1.5707963267948966 3.141592653589793 3.141592653589793 -> xyz=-0.20 -0.05 0 rpy=1.5707963267948966 3.141592653589793 1.5707963267948966

Commit message: update

File: orthrus_interfaces/models/orthrus/urdf/orthrus.urdf (robot description, URDF)
Before this commit: robot orthrus, 17 links, 16 joints
Links:
- link LF_HAA_link: geometry collision mesh filename=file:////home/orthrus/orthrus/install/orthrus_interfaces/sh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; visual mesh filename=file:////home/orthrus/orthrus/install/orthrus_interfaces/sh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
- link LF_HFE_link: geometry collision mesh filename=file:////home/orthrus/orthrus/install/orthrus_interfaces/sh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; visual mesh filename=file:////home/orthrus/orthrus/install/orthrus_interfaces/sh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
- link LF_KFE_link: geometry collision mesh filename=file:////home/orthrus/orthrus/install/orthrus_interfaces/sh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; visual mesh filename=file:////home/orthrus/orthrus/install/orthrus_interfaces/sh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
- link LH_HAA_link: geometry collision mesh filename=file:////home/orthrus/orthrus/install/orthrus_interfaces/sh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; visual mesh filename=file:////home/orthrus/orthrus/install/orthrus_interfaces/sh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
- link LH_HFE_link: geometry collision mesh filename=file:////home/orthrus/orthrus/install/orthrus_interfaces/sh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; visual mesh filename=file:////home/orthrus/orthrus/install/orthrus_interfaces/sh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
- link LH_KFE_link: geometry collision mesh filename=file:////home/orthrus/orthrus/install/orthrus_interfaces/sh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; visual mesh filename=file:////home/orthrus/orthrus/install/orthrus_interfaces/sh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
- link RF_HAA_link: geometry collision mesh filename=file:////home/orthrus/orthrus/install/orthrus_interfaces/sh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; visual mesh filename=file:////home/orthrus/orthrus/install/orthrus_interfaces/sh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
- link RF_HFE_link: geometry collision mesh filename=file:////home/orthrus/orthrus/install/orthrus_interfaces/sh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; visual mesh filename=file:////home/orthrus/orthrus/install/orthrus_interfaces/sh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
- link RF_KFE_link: geometry collision mesh filename=file:////home/orthrus/orthrus/install/orthrus_interfaces/sh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; visual mesh filename=file:////home/orthrus/orthrus/install/orthrus_interfaces/sh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
- link RH_HAA_link: geometry collision mesh filename=file:////home/orthrus/orthrus/install/orthrus_interfaces/sh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; visual mesh filename=file:////home/orthrus/orthrus/install/orthrus_interfaces/sh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
- link RH_HFE_link: geometry collision mesh filename=file:////home/orthrus/orthrus/install/orthrus_interfaces/sh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; visual mesh filename=file:////home/orthrus/orthrus/install/orthrus_interfaces/sh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
- link RH_KFE_link: geometry collision mesh filename=file:////home/orthrus/orthrus/install/orthrus_interfaces/sh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; visual mesh filename=file:////home/orthrus/orthrus/install/orthrus_interfaces/sh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
- link base: geometry collision mesh filename=file:////home/orthrus/orthrus/install/orthrus_interfaces/sh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; visual mesh filename=file:////home/orthrus/orthrus/install/orthrus_interfaces/sh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

File: orthrus_interfaces/models/orthrus/urdf/orthrus.urdf.xacro (robot description, xacro)
@@ -61,5 +61,5 @@
   <gazebo>
     <plugin filename="libgazebo_ros2_control.so" name="gazebo_ros2_control">
-      <parameters>/home/evence/code_file/ros2_ws/orthrus/src/orthrus_ros2_pack/orthrus_sim/orthrus_gazebo/config/orthrus.yaml</parameters>
+      <parameters>/home/orthrus/orthrus/src/orthrus_ros2_pack/orthrus_sim/orthrus_gazebo/config/orthrus.yaml</parameters>
     </plugin>
   </gazebo>
