Commit message: update

File: orthrus_interfaces/models/orthrus/urdf/orthrus.urdf (robot description, URDF)
Before this commit: robot orthrus, 17 links, 16 joints
Links:
- link LF_HAA_link: geometry collision mesh filename=file:////home/orthrus/orthrus/install/orthrus_interfaces/sh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; visual mesh filename=file:////home/orthrus/orthrus/install/orthrus_interfaces/sh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
- link LF_HFE_link: geometry collision mesh filename=file:////home/orthrus/orthrus/install/orthrus_interfaces/sh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; visual mesh filename=file:////home/orthrus/orthrus/install/orthrus_interfaces/sh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
- link LF_KFE_link: geometry collision mesh filename=file:////home/orthrus/orthrus/install/orthrus_interfaces/sh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; visual mesh filename=file:////home/orthrus/orthrus/install/orthrus_interfaces/sh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
- link LH_HAA_link: geometry collision mesh filename=file:////home/orthrus/orthrus/install/orthrus_interfaces/sh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; visual mesh filename=file:////home/orthrus/orthrus/install/orthrus_interfaces/sh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
- link LH_HFE_link: geometry collision mesh filename=file:////home/orthrus/orthrus/install/orthrus_interfaces/sh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; visual mesh filename=file:////home/orthrus/orthrus/install/orthrus_interfaces/sh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
- link LH_KFE_link: geometry collision mesh filename=file:////home/orthrus/orthrus/install/orthrus_interfaces/sh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; visual mesh filename=file:////home/orthrus/orthrus/install/orthrus_interfaces/sh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
- link RF_HAA_link: geometry collision mesh filename=file:////home/orthrus/orthrus/install/orthrus_interfaces/sh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; visual mesh filename=file:////home/orthrus/orthrus/install/orthrus_interfaces/sh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
- link RF_HFE_link: geometry collision mesh filename=file:////home/orthrus/orthrus/install/orthrus_interfaces/sh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; visual mesh filename=file:////home/orthrus/orthrus/install/orthrus_interfaces/sh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
- link RF_KFE_link: geometry collision mesh filename=file:////home/orthrus/orthrus/install/orthrus_interfaces/sh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; visual mesh filename=file:////home/orthrus/orthrus/install/orthrus_interfaces/sh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
- link RH_HAA_link: geometry collision mesh filename=file:////home/orthrus/orthrus/install/orthrus_interfaces/sh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; visual mesh filename=file:////home/orthrus/orthrus/install/orthrus_interfaces/sh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
- link RH_HFE_link: geometry collision mesh filename=file:////home/orthrus/orthrus/install/orthrus_interfaces/sh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; visual mesh filename=file:////home/orthrus/orthrus/install/orthrus_interfaces/sh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
- link RH_KFE_link: geometry collision mesh filename=file:////home/orthrus/orthrus/install/orthrus_interfaces/sh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; visual mesh filename=file:////home/orthrus/orthrus/install/orthrus_interfaces/sh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
- link base: mass 7 -> 4.429; geometry collision mesh filename=file:////home/orthrus/orthrus/install/orthrus_interfaces/sh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; visual mesh filename=file:////home/orthrus/orthrus/install/orthrus_interfaces/sh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

File: orthrus_interfaces/models/orthrus/urdf/orthrus_gazebo.urdf (robot description, URDF)
Before this commit: robot orthrus, 17 links, 16 joints
Links:
- link LF_HAA_link: geometry collision mesh filename=file:////home/orthrus/orthrus/install/orthrus_interfaces/sh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; visual mesh filename=file:////home/orthrus/orthrus/install/orthrus_interfaces/sh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
- link LF_HFE_link: geometry collision mesh filename=file:////home/orthrus/orthrus/install/orthrus_interfaces/sh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; visual mesh filename=file:////home/orthrus/orthrus/install/orthrus_interfaces/sh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
- link LF_KFE_link: geometry collision mesh filename=file:////home/orthrus/orthrus/install/orthrus_interfaces/sh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; visual mesh filename=file:////home/orthrus/orthrus/install/orthrus_interfaces/sh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
- link LH_HAA_link: geometry collision mesh filename=file:////home/orthrus/orthrus/install/orthrus_interfaces/sh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; visual mesh filename=file:////home/orthrus/orthrus/install/orthrus_interfaces/sh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
- link LH_HFE_link: geometry collision mesh filename=file:////home/orthrus/orthrus/install/orthrus_interfaces/sh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; visual mesh filename=file:////home/orthrus/orthrus/install/orthrus_interfaces/sh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
- link LH_KFE_link: geometry collision mesh filename=file:////home/orthrus/orthrus/install/orthrus_interfaces/sh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; visual mesh filename=file:////home/orthrus/orthrus/install/orthrus_interfaces/sh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
- link RF_HAA_link: geometry collision mesh filename=file:////home/orthrus/orthrus/install/orthrus_interfaces/sh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; visual mesh filename=file:////home/orthrus/orthrus/install/orthrus_interfaces/sh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
- link RF_HFE_link: geometry collision mesh filename=file:////home/orthrus/orthrus/install/orthrus_interfaces/sh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; visual mesh filename=file:////home/orthrus/orthrus/install/orthrus_interfaces/sh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
- link RF_KFE_link: geometry collision mesh filename=file:////home/orthrus/orthrus/install/orthrus_interfaces/sh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; visual mesh filename=file:////home/orthrus/orthrus/install/orthrus_interfaces/sh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
- link RH_HAA_link: geometry collision mesh filename=file:////home/orthrus/orthrus/install/orthrus_interfaces/sh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; visual mesh filename=file:////home/orthrus/orthrus/install/orthrus_interfaces/sh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
- link RH_HFE_link: geometry collision mesh filename=file:////home/orthrus/orthrus/install/orthrus_interfaces/sh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; visual mesh filename=file:////home/orthrus/orthrus/install/orthrus_interfaces/sh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
- link RH_KFE_link: geometry collision mesh filename=file:////home/orthrus/orthrus/install/orthrus_interfaces/sh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; visual mesh filename=file:////home/orthrus/orthrus/install/orthrus_interfaces/sh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
- link base: mass 7 -> 4.429; geometry collision mesh filename=file:////home/orthrus/orthrus/install/orthrus_interfaces/sh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; visual mesh filename=file:////home/orthrus/orthrus/install/orthrus_interfaces/sh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

File: orthrus_interfaces/models/orthrus/urdf/orthrus_real.urdf (robot description, URDF)
Before this commit: robot orthrus, 17 links, 16 joints
Links:
- link LF_HAA_link: geometry collision mesh filename=file:////home/orthrus/orthrus/install/orthrus_interfaces/sh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; visual mesh filename=file:////home/orthrus/orthrus/install/orthrus_interfaces/sh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
- link LF_HFE_link: geometry collision mesh filename=file:////home/orthrus/orthrus/install/orthrus_interfaces/sh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; visual mesh filename=file:////home/orthrus/orthrus/install/orthrus_interfaces/sh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
- link LF_KFE_link: geometry collision mesh filename=file:////home/orthrus/orthrus/install/orthrus_interfaces/sh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; visual mesh filename=file:////home/orthrus/orthrus/install/orthrus_interfaces/sh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
- link LH_HAA_link: geometry collision mesh filename=file:////home/orthrus/orthrus/install/orthrus_interfaces/sh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; visual mesh filename=file:////home/orthrus/orthrus/install/orthrus_interfaces/sh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
- link LH_HFE_link: geometry collision mesh filename=file:////home/orthrus/orthrus/install/orthrus_interfaces/sh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; visual mesh filename=file:////home/orthrus/orthrus/install/orthrus_interfaces/sh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
- link LH_KFE_link: geometry collision mesh filename=file:////home/orthrus/orthrus/install/orthrus_interfaces/sh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; visual mesh filename=file:////home/orthrus/orthrus/install/orthrus_interfaces/sh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
- link RF_HAA_link: geometry collision mesh filename=file:////home/orthrus/orthrus/install/orthrus_interfaces/sh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; visual mesh filename=file:////home/orthrus/orthrus/install/orthrus_interfaces/sh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
- link RF_HFE_link: geometry collision mesh filename=file:////home/orthrus/orthrus/install/orthrus_interfaces/sh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; visual mesh filename=file:////home/orthrus/orthrus/install/orthrus_interfaces/sh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
- link RF_KFE_link: geometry collision mesh filename=file:////home/orthrus/orthrus/install/orthrus_interfaces/sh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; visual mesh filename=file:////home/orthrus/orthrus/install/orthrus_interfaces/sh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
- link RH_HAA_link: geometry collision mesh filename=file:////home/orthrus/orthrus/install/orthrus_interfaces/sh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; visual mesh filename=file:////home/orthrus/orthrus/install/orthrus_interfaces/sh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
- link RH_HFE_link: geometry collision mesh filename=file:////home/orthrus/orthrus/install/orthrus_interfaces/sh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; visual mesh filename=file:////home/orthrus/orthrus/install/orthrus_interfaces/sh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
- link RH_KFE_link: geometry collision mesh filename=file:////home/orthrus/orthrus/install/orthrus_interfaces/sh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; visual mesh filename=file:////home/orthrus/orthrus/install/orthrus_interfaces/sh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
- link base: mass 7 -> 4.429; geometry collision mesh filename=file:////home/orthrus/orthrus/install/orthrus_interfaces/sh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; visual mesh filename=file:////home/orthrus/orthrus/install/orthrus_interfaces/sh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

Commit message: update

File: orthrus_interfaces/models/orthrus/urdf/orthrus.urdf (robot description, URDF)
Before this commit: robot orthrus, 17 links, 16 joints
Links:
- link LF_HAA_link: mass 0.7 -> 0.67; geometry collision mesh filename=file:////home/evence/code_file/ros2_ws/orthrus/install/orth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; visual mesh filename=file:////home/evence/code_file/ros2_ws/orthrus/install/orth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
- link LF_HFE_link: mass 1 -> 0.928; geometry collision mesh filename=file:////home/evence/code_file/ros2_ws/orthrus/install/orth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; visual mesh filename=file:////home/evence/code_file/ros2_ws/orthrus/install/orth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
- link LF_KFE_link: mass 0.2 -> 0.187; geometry collision mesh filename=file:////home/evence/code_file/ros2_ws/orthrus/install/orth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; visual mesh filename=file:////home/evence/code_file/ros2_ws/orthrus/install/orth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
- link LH_HAA_link: mass 0.7 -> 0.67; geometry collision mesh filename=file:////home/evence/code_file/ros2_ws/orthrus/install/orth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; visual mesh filename=file:////home/evence/code_file/ros2_ws/orthrus/install/orth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
- link LH_HFE_link: mass 1 -> 0.928; geometry collision mesh filename=file:////home/evence/code_file/ros2_ws/orthrus/install/orth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; visual mesh filename=file:////home/evence/code_file/ros2_ws/orthrus/install/orth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
- link LH_KFE_link: mass 0.2 -> 0.187; geometry collision mesh filename=file:////home/evence/code_file/ros2_ws/orthrus/install/orth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; visual mesh filename=file:////home/evence/code_file/ros2_ws/orthrus/install/orth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
- link RF_HAA_link: mass 0.7 -> 0.67; geometry collision mesh filename=file:////home/evence/code_file/ros2_ws/orthrus/install/orth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; visual mesh filename=file:////home/evence/code_file/ros2_ws/orthrus/install/orth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
- link RF_HFE_link: mass 1 -> 0.928; geometry collision mesh filename=file:////home/evence/code_file/ros2_ws/orthrus/install/orth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; visual mesh filename=file:////home/evence/code_file/ros2_ws/orthrus/install/orth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
- link RF_KFE_link: mass 0.2 -> 0.187; geometry collision mesh filename=file:////home/evence/code_file/ros2_ws/orthrus/install/orth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; visual mesh filename=file:////home/evence/code_file/ros2_ws/orthrus/install/orth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
- link RH_HAA_link: mass 0.7 -> 0.67; geometry collision mesh filename=file:////home/evence/code_file/ros2_ws/orthrus/install/orth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; visual mesh filename=file:////home/evence/code_file/ros2_ws/orthrus/install/orth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
- link RH_HFE_link: mass 1 -> 0.928; geometry collision mesh filename=file:////home/evence/code_file/ros2_ws/orthrus/install/orth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; visual mesh filename=file:////home/evence/code_file/ros2_ws/orthrus/install/orth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
- link RH_KFE_link: mass 0.2 -> 0.187; geometry collision mesh filename=file:////home/evence/code_file/ros2_ws/orthrus/install/orth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; visual mesh filename=file:////home/evence/code_file/ros2_ws/orthrus/install/orth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
- link base: geometry collision mesh filename=file:////home/evence/code_file/ros2_ws/orthrus/install/orth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; visual mesh filename=file:////home/evence/code_file/ros2_ws/orthrus/install/orth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

File: orthrus_interfaces/models/orthrus/urdf/orthrus_gazebo.urdf (robot description, URDF)
Before this commit: robot orthrus, 17 links, 16 joints
Links:
- link LF_HAA_link: mass 0.7 -> 0.67; geometry collision mesh filename=file:////home/evence/code_file/ros2_ws/orthrus/install/orth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; visual mesh filename=file:////home/evence/code_file/ros2_ws/orthrus/install/orth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
- link LF_HFE_link: mass 1 -> 0.928; geometry collision mesh filename=file:////home/evence/code_file/ros2_ws/orthrus/install/orth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; visual mesh filename=file:////home/evence/code_file/ros2_ws/orthrus/install/orth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
- link LF_KFE_link: mass 0.2 -> 0.187; geometry collision mesh filename=file:////home/evence/code_file/ros2_ws/orthrus/install/orth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; visual mesh filename=file:////home/evence/code_file/ros2_ws/orthrus/install/orth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
- link LH_HAA_link: mass 0.7 -> 0.67; geometry collision mesh filename=file:////home/evence/code_file/ros2_ws/orthrus/install/orth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; visual mesh filename=file:////home/evence/code_file/ros2_ws/orthrus/install/orth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
- link LH_HFE_link: mass 1 -> 0.928; geometry collision mesh filename=file:////home/evence/code_file/ros2_ws/orthrus/install/orth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; visual mesh filename=file:////home/evence/code_file/ros2_ws/orthrus/install/orth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
- link LH_KFE_link: mass 0.2 -> 0.187; geometry collision mesh filename=file:////home/evence/code_file/ros2_ws/orthrus/install/orth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; visual mesh filename=file:////home/evence/code_file/ros2_ws/orthrus/install/orth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
- link RF_HAA_link: mass 0.7 -> 0.67; geometry collision mesh filename=file:////home/evence/code_file/ros2_ws/orthrus/install/orth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; visual mesh filename=file:////home/evence/code_file/ros2_ws/orthrus/install/orth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
- link RF_HFE_link: mass 1 -> 0.928; geometry collision mesh filename=file:////home/evence/code_file/ros2_ws/orthrus/install/orth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; visual mesh filename=file:////home/evence/code_file/ros2_ws/orthrus/install/orth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
- link RF_KFE_link: mass 0.2 -> 0.187; geometry collision mesh filename=file:////home/evence/code_file/ros2_ws/orthrus/install/orth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; visual mesh filename=file:////home/evence/code_file/ros2_ws/orthrus/install/orth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
- link RH_HAA_link: mass 0.7 -> 0.67; geometry collision mesh filename=file:////home/evence/code_file/ros2_ws/orthrus/install/orth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; visual mesh filename=file:////home/evence/code_file/ros2_ws/orthrus/install/orth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
- link RH_HFE_link: mass 1 -> 0.928; geometry collision mesh filename=file:////home/evence/code_file/ros2_ws/orthrus/install/orth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; visual mesh filename=file:////home/evence/code_file/ros2_ws/orthrus/install/orth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
- link RH_KFE_link: mass 0.2 -> 0.187; geometry collision mesh filename=file:////home/evence/code_file/ros2_ws/orthrus/install/orth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; visual mesh filename=file:////home/evence/code_file/ros2_ws/orthrus/install/orth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
- link base: geometry collision mesh filename=file:////home/evence/code_file/ros2_ws/orthrus/install/orth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; visual mesh filename=file:////home/evence/code_file/ros2_ws/orthrus/install/orth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

File: orthrus_interfaces/models/orthrus/urdf/orthrus_real.urdf (robot description, URDF)
Before this commit: robot orthrus, 17 links, 16 joints
Links:
- link LF_HAA_link: mass 0.7 -> 0.67; geometry collision mesh filename=file:////home/evence/code_file/ros2_ws/orthrus/install/orth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; visual mesh filename=file:////home/evence/code_file/ros2_ws/orthrus/install/orth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
- link LF_HFE_link: mass 1 -> 0.928; geometry collision mesh filename=file:////home/evence/code_file/ros2_ws/orthrus/install/orth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; visual mesh filename=file:////home/evence/code_file/ros2_ws/orthrus/install/orth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
- link LF_KFE_link: mass 0.2 -> 0.187; geometry collision mesh filename=file:////home/evence/code_file/ros2_ws/orthrus/install/orth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; visual mesh filename=file:////home/evence/code_file/ros2_ws/orthrus/install/orth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
- link LH_HAA_link: mass 0.7 -> 0.67; geometry collision mesh filename=file:////home/evence/code_file/ros2_ws/orthrus/install/orth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; visual mesh filename=file:////home/evence/code_file/ros2_ws/orthrus/install/orth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
- link LH_HFE_link: mass 1 -> 0.928; geometry collision mesh filename=file:////home/evence/code_file/ros2_ws/orthrus/install/orth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; visual mesh filename=file:////home/evence/code_file/ros2_ws/orthrus/install/orth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
- link LH_KFE_link: mass 0.2 -> 0.187; geometry collision mesh filename=file:////home/evence/code_file/ros2_ws/orthrus/install/orth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; visual mesh filename=file:////home/evence/code_file/ros2_ws/orthrus/install/orth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
- link RF_HAA_link: mass 0.7 -> 0.67; geometry collision mesh filename=file:////home/evence/code_file/ros2_ws/orthrus/install/orth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; visual mesh filename=file:////home/evence/code_file/ros2_ws/orthrus/install/orth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
- link RF_HFE_link: mass 1 -> 0.928; geometry collision mesh filename=file:////home/evence/code_file/ros2_ws/orthrus/install/orth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; visual mesh filename=file:////home/evence/code_file/ros2_ws/orthrus/install/orth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
- link RF_KFE_link: mass 0.2 -> 0.187; geometry collision mesh filename=file:////home/evence/code_file/ros2_ws/orthrus/install/orth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; visual mesh filename=file:////home/evence/code_file/ros2_ws/orthrus/install/orth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
- link RH_HAA_link: mass 0.7 -> 0.67; geometry collision mesh filename=file:////home/evence/code_file/ros2_ws/orthrus/install/orth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; visual mesh filename=file:////home/evence/code_file/ros2_ws/orthrus/install/orth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
- link RH_HFE_link: mass 1 -> 0.928; geometry collision mesh filename=file:////home/evence/code_file/ros2_ws/orthrus/install/orth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; visual mesh filename=file:////home/evence/code_file/ros2_ws/orthrus/install/orth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
- link RH_KFE_link: mass 0.2 -> 0.187; geometry collision mesh filename=file:////home/evence/code_file/ros2_ws/orthrus/install/orth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; visual mesh filename=file:////home/evence/code_file/ros2_ws/orthrus/install/orth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
- link base: geometry collision mesh filename=file:////home/evence/code_file/ros2_ws/orthrus/install/orth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; visual mesh filename=file:////home/evence/code_file/ros2_ws/orthrus/install/orth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

Commit message: update

File: orthrus_interfaces/models/orthrus/urdf/orthrus.urdf (robot description, URDF)
Before this commit: robot orthrus, 17 links, 16 joints
Links:
- link LF_HAA_link: mass 0.7 -> 0.67
- link LF_HFE_link: mass 1 -> 0.928
- link LF_KFE_link: mass 0.2 -> 0.187
- link LH_HAA_link: mass 0.7 -> 0.67
- link LH_HFE_link: mass 1 -> 0.928
- link LH_KFE_link: mass 0.2 -> 0.187
- link RF_HAA_link: mass 0.7 -> 0.67
- link RF_HFE_link: mass 1 -> 0.928
- link RF_KFE_link: mass 0.2 -> 0.187
- link RH_HAA_link: mass 0.7 -> 0.67
- link RH_HFE_link: mass 1 -> 0.928
- link RH_KFE_link: mass 0.2 -> 0.187

File: orthrus_interfaces/models/orthrus/urdf/orthrus_gazebo.urdf (robot description, URDF)
Before this commit: robot orthrus, 17 links, 16 joints
Links:
- link LF_HAA_link: mass 0.7 -> 0.67
- link LF_HFE_link: mass 1 -> 0.928
- link LF_KFE_link: mass 0.2 -> 0.187
- link LH_HAA_link: mass 0.7 -> 0.67
- link LH_HFE_link: mass 1 -> 0.928
- link LH_KFE_link: mass 0.2 -> 0.187
- link RF_HAA_link: mass 0.7 -> 0.67
- link RF_HFE_link: mass 1 -> 0.928
- link RF_KFE_link: mass 0.2 -> 0.187
- link RH_HAA_link: mass 0.7 -> 0.67
- link RH_HFE_link: mass 1 -> 0.928
- link RH_KFE_link: mass 0.2 -> 0.187

File: orthrus_interfaces/models/orthrus/urdf/orthrus_real.urdf (robot description, URDF)
Before this commit: robot orthrus, 17 links, 16 joints
Links:
- link LF_HAA_link: mass 0.7 -> 0.67
- link LF_HFE_link: mass 1 -> 0.928
- link LF_KFE_link: mass 0.2 -> 0.187
- link LH_HAA_link: mass 0.7 -> 0.67
- link LH_HFE_link: mass 1 -> 0.928
- link LH_KFE_link: mass 0.2 -> 0.187
- link RF_HAA_link: mass 0.7 -> 0.67
- link RF_HFE_link: mass 1 -> 0.928
- link RF_KFE_link: mass 0.2 -> 0.187
- link RH_HAA_link: mass 0.7 -> 0.67
- link RH_HFE_link: mass 1 -> 0.928
- link RH_KFE_link: mass 0.2 -> 0.187
