Commit message: update

File: orthrus_description/models/orthrus/urdf/orthrus.urdf.xacro (robot description, xacro)
@@ -2,5 +2,5 @@
 <robot name="orthrus"
   xmlns:xacro="http://ros.org/wiki/xacro">
-  <xacro:property name="meshes_folder" value="file:///$(find orthrus_interfaces)/models/orthrus/meshes" />
+  <xacro:property name="meshes_folder" value="file:///$(find orthrus_description)/models/orthrus/meshes" />
   <xacro:property name="orthrus_config_path" value="file:///$(find orthrus_gazebo)/config/orthrus.yaml" />
   <xacro:include filename="orthrus_base.xacro"/>

File: orthrus_description/models/orthrus/urdf/orthrus_gazebo.urdf.xacro (robot description, xacro)
@@ -1,5 +1,5 @@
 <robot name="orthrus"
   xmlns:xacro="http://ros.org/wiki/xacro">
-  <xacro:property name="meshes_folder" value="file:///$(find orthrus_interfaces)/models/orthrus/meshes" />
+  <xacro:property name="meshes_folder" value="file:///$(find orthrus_description)/models/orthrus/meshes" />
   <xacro:property name="orthrus_config_path" value="file:///$(find orthrus_gazebo)/config/orthrus.yaml" />
   <xacro:include filename="orthrus_base.xacro"/>

File: orthrus_description/models/orthrus/urdf/orthrus_real.urdf.xacro (robot description, xacro)
@@ -2,5 +2,5 @@
 <robot name="orthrus"
   xmlns:xacro="http://ros.org/wiki/xacro">
-  <xacro:property name="meshes_folder" value="file:///$(find orthrus_interfaces)/models/orthrus/meshes" />
+  <xacro:property name="meshes_folder" value="file:///$(find orthrus_description)/models/orthrus/meshes" />
   <xacro:property name="orthrus_config_path" value="file:///$(find orthrus_control)/config/orthrus.yaml" />
   <xacro:include filename="orthrus_base.xacro"/>
